Commit message: swap to estimated inertias to troubleshoot

File: src/catbot_description/urdf/catbot/catbot_macro.xacro (robot description, xacro)
@@ -2,4 +2,5 @@
 <robot xmlns:xacro="http://wiki.ros.org/xacro">
   <xacro:macro name="catbot" params="prefix parent *origin">
+    <xacro:include filename="inertial_macros.xacro"/>
     <!-- base_joint fixes base_link to the environment -->
     <joint name="${prefix}base_joint" type="fixed">
@@ -30,15 +31,5 @@
         </geometry>
       </collision>
-      <inertial>
-        <origin xyz="0.00027961412402240787278 0.0046876789374875821662 -0.0054409557585405705568"
-        rpy="0 0 0" />
-        <mass value="1.015668141636539179" />
-        <inertia ixx="0.0065127126032337098738"
-        ixy="1.5566438777546685336e-07"
-        ixz="3.6708728527239311778e-06"
-        iyy="0.0025991819436423468752"
-        iyz="6.1954470337197611722e-05"
-        izz="0.0071648278899316356766" />
-      </inertial>
+      <xacro:chassis_inertia/>
     </link>
     <link name="wheel_assm">
@@ -58,15 +49,5 @@
         </geometry>
       </collision>
-      <inertial>
-        <origin xyz="2.5876683183573441879e-09 -2.5321947361304500679e-09 -0.0043217676979120569353"
-        rpy="0 0 0" />
-        <mass value="0.054377782220193432439" />
-        <inertia ixx="1.7947780629583346784e-05"
-        ixy="-3.8234084819748992999e-12"
-        ixz="-1.6934852924892931359e-12"
-        iyy="1.7621269066491268497e-05"
-        iyz="-2.0136050748759971485e-12"
-        izz="2.8213568549230894094e-05" />
-      </inertial>
+      <xacro:wheel_inertia/>
     </link>
     <joint name="rr_wheel" type="continuous">
@@ -95,15 +76,5 @@
         </geometry>
       </collision>
-      <inertial>
-        <origin xyz="2.5876683388231371246e-09 -2.5321947856343332086e-09 -0.004321767697912089895"
-        rpy="0 0 0" />
-        <mass value="0.054377782220193432439" />
-        <inertia ixx="1.7947780629583370501e-05"
-        ixy="-3.8234084811821872389e-12"
-        ixz="-1.6934852959410392741e-12"
-        iyy="1.7621269066491275274e-05"
-        iyz="-2.013605069932675335e-12"
-        izz="2.8213568549230904259e-05" />
-      </inertial>
+      <xacro:wheel_inertia/>
     </link>
     <joint name="rf_wheel" type="continuous">
@@ -132,15 +103,5 @@
         </geometry>
       </collision>
-      <inertial>
-        <origin xyz="2.5876683494035538817e-09 -2.5321947903698363363e-09 -0.0043217676979121003034"
-        rpy="0 0 0" />
-        <mass value="0.054377782220193432439" />
-        <inertia ixx="1.7947780629583370501e-05"
-        ixy="-3.8234084811821831999e-12"
-        ixz="-1.6934852949411820834e-12"
-        iyy="1.7621269066491278662e-05"
-        iyz="-2.0136050682372531551e-12"
-        izz="2.8213568549230904259e-05" />
-      </inertial>
+      <xacro:wheel_inertia/>
     </link>
     <joint name="rl_wheel" type="continuous">
@@ -169,15 +130,5 @@
         </geometry>
       </collision>
-      <inertial>
-        <origin xyz="2.587668269624447972e-09 -2.5321945322547953329e-09 -0.0043217676979121323957"
-        rpy="0 0 0" />
-        <mass value="0.054377782220193432439" />
-        <inertia ixx="1.7947780629583373889e-05"
-        ixy="-3.8234084825756295263e-12"
-        ixz="-1.6934852991867637216e-12"
-        iyy="1.7621269066491278662e-05"
-        iyz="-2.0136050681091290175e-12"
-        izz="2.8213568549230907647e-05" />
-      </inertial>
+      <xacro:wheel_inertia/>
     </link>
     <joint name="fl_wheel" type="continuous">

Commit message: swapped to fixed rear wheels for testing

File: src/catbot_description/urdf/catbot/catbot_macro.xacro (robot description, xacro)
@@ -44,5 +44,5 @@
     <xacro:wheel_inertia/>
   </link>
-  <joint name="rr_wheel" type="continuous">
+  <joint name="rr_wheel" type="fixed">
     <origin xyz="-0.077614131532514007983 0.080478921592024327269 -0.030500000000000013212"
     rpy="-1.570796326794896558 0.67540343776289657463 -1.5707963267948956698" />
@@ -50,6 +50,6 @@
     <child link="wheel_assm" />
     <axis xyz="0 0 1" />
-    <limit effort="1" velocity="20" />
-    <joint_properties friction="0.0" />
+    <!-- <limit effort="1" velocity="20" />
+    <joint_properties friction="0.0" /> -->
   </joint>
   <link name="wheel_assm_2">
@@ -98,5 +98,5 @@
     <xacro:wheel_inertia/>
   </link>
-  <joint name="rl_wheel" type="continuous">
+  <joint name="rl_wheel" type="fixed">
     <origin xyz="0.078385868467483257871 0.080478921592024507681 -0.030500000000000044437"
     rpy="-1.570796326794896558 -5.0445758681405660746e-15 1.5707963267948970021" />
@@ -104,6 +104,6 @@
     <child link="wheel_assm_3" />
     <axis xyz="0 0 1" />
-    <limit effort="1" velocity="20" />
-    <joint_properties friction="0.0" />
+    <!-- <limit effort="1" velocity="20" />
+    <joint_properties friction="0.0" /> -->
   </joint>
   <link name="wheel_assm_4">

File: src/catbot_description/urdf/catbot/inertial_macros.xacro (robot description, xacro)
@@ -45,5 +45,5 @@
     <xacro:property name="chassis_height" value="0.105"/>
     <xacro:macro name="chassis_inertia">
-        <xacro:inertial_box mass="${chassis_mass}" x="${chassis_length}" y="${chassis_width}" z="${chassis_height}">
+        <xacro:inertial_box mass="0.5" x="${chassis_length}" y="${chassis_width}" z="${chassis_height}">
             <origin xyz="${chassis_length/2} 0 ${chassis_height/2}" rpy="0 0 0"/>
         </xacro:inertial_box>

Commit message: works FWD!

File: src/catbot_description/urdf/catbot/catbot_macro.xacro (robot description, xacro)
@@ -24,5 +24,15 @@
       </geometry>
     </collision>
-    <xacro:chassis_inertia/>
+     <inertial>
+        <origin xyz="0.00027961412402240787278 0.0046876789374875821662 -0.0054409557585405705568"
+        rpy="0 0 0" />
+        <mass value="1.015668141636539179" />
+        <inertia ixx="0.0065127126032337098738"
+        ixy="1.5566438777546685336e-07"
+        ixz="3.6708728527239311778e-06"
+        iyy="0.0025991819436423468752"
+        iyz="6.1954470337197611722e-05"
+        izz="0.0071648278899316356766" />
+      </inertial>
   </link>
   <link name="wheel_assm">
@@ -130,5 +140,5 @@
     <parent link="still_chassis_assm" />
     <child link="wheel_assm_4" />
-    <axis xyz="0 0 1" />
+    <axis xyz="0 0 -1" />
     <limit effort="1" velocity="20" />
     <joint_properties friction="0.0" />

Commit message: return to using Onshape inertias!

File: src/catbot_description/urdf/catbot/catbot_macro.xacro (robot description, xacro)
@@ -52,5 +52,15 @@
       </geometry>
     </collision>
-    <xacro:wheel_inertia/>
+    <inertial>
+      <origin xyz="2.5876683183573441879e-09 -2.5321947361304500679e-09 -0.0043217676979120569353"
+      rpy="0 0 0" />
+      <mass value="0.054377782220193432439" />
+      <inertia ixx="1.7947780629583346784e-05"
+      ixy="-3.8234084819748992999e-12"
+      ixz="-1.6934852924892931359e-12"
+      iyy="1.7621269066491268497e-05"
+      iyz="-2.0136050748759971485e-12"
+      izz="2.8213568549230894094e-05" />
+      </inertial>
   </link>
   <joint name="rr_wheel" type="fixed">
@@ -79,5 +89,15 @@
       </geometry>
     </collision>
-    <xacro:wheel_inertia/>
+    <inertial>
+      <origin xyz="2.5876683388231371246e-09 -2.5321947856343332086e-09 -0.004321767697912089895"
+      rpy="0 0 0" />
+      <mass value="0.054377782220193432439" />
+      <inertia ixx="1.7947780629583370501e-05"
+      ixy="-3.8234084811821872389e-12"
+      ixz="-1.6934852959410392741e-12"
+      iyy="1.7621269066491275274e-05"
+      iyz="-2.013605069932675335e-12"
+      izz="2.8213568549230904259e-05" />
+    </inertial>
   </link>
   <joint name="rf_wheel" type="continuous">
@@ -106,5 +126,15 @@
       </geometry>
     </collision>
-    <xacro:wheel_inertia/>
+    <inertial>
+      <origin xyz="2.5876683494035538817e-09 -2.5321947903698363363e-09 -0.0043217676979121003034"
+      rpy="0 0 0" />
+      <mass value="0.054377782220193432439" />
+      <inertia ixx="1.7947780629583370501e-05"
+      ixy="-3.8234084811821831999e-12"
+      ixz="-1.6934852949411820834e-12"
+      iyy="1.7621269066491278662e-05"
+      iyz="-2.0136050682372531551e-12"
+      izz="2.8213568549230904259e-05" />
+    </inertial>
   </link>
   <joint name="rl_wheel" type="fixed">
@@ -133,5 +163,15 @@
       </geometry>
     </collision>
-    <xacro:wheel_inertia/>
+    <inertial>
+      <origin xyz="2.587668269624447972e-09 -2.5321945322547953329e-09 -0.0043217676979121323957"
+      rpy="0 0 0" />
+      <mass value="0.054377782220193432439" />
+      <inertia ixx="1.7947780629583373889e-05"
+      ixy="-3.8234084825756295263e-12"
+      ixz="-1.6934852991867637216e-12"
+      iyy="1.7621269066491278662e-05"
+      iyz="-2.0136050681091290175e-12"
+      izz="2.8213568549230907647e-05" />
+    </inertial>
   </link>
   <joint name="fl_wheel" type="continuous">

Commit message: approximate wheel collision as spheres

File: src/catbot_description/urdf/catbot/catbot_macro.xacro (robot description, xacro)
@@ -2,4 +2,5 @@
 <robot xmlns:xacro="http://wiki.ros.org/xacro">
   <xacro:include filename="inertial_macros.xacro"/>
+  <xacro:property name="sphere_wheel_offset" value="0.006"/>
   <link name="base_link"></link>
   <joint name="chassis_joint" type="fixed">
@@ -47,7 +48,8 @@
     </visual>
     <collision>
-      <origin xyz="0 0 0" rpy="0 -0 0" />
+      <origin xyz="0 0 -${sphere_wheel_offset}" rpy="0 -0 0" />
       <geometry>
-        <mesh filename="package://catbot_description/meshes/collision/wheel_assm_collision.stl" />
+        <!-- <mesh filename="package://catbot_description/meshes/collision/wheel_assm_collision.stl" /> -->
+        <sphere radius="${wheel_radius}"/>
       </geometry>
     </collision>
@@ -84,7 +86,8 @@
     </visual>
     <collision>
-      <origin xyz="0 0 0" rpy="0 -0 0" />
+      <origin xyz="0 0 -${sphere_wheel_offset}" rpy="0 -0 0" />
       <geometry>
-        <mesh filename="package://catbot_description/meshes/collision/wheel_assm_2_collision.stl" />
+        <!-- <mesh filename="package://catbot_description/meshes/collision/wheel_assm_2_collision.stl" /> -->
+        <sphere radius="${wheel_radius}"/>
       </geometry>
     </collision>
@@ -121,7 +124,8 @@
     </visual>
     <collision>
-      <origin xyz="0 0 0" rpy="0 -0 0" />
+      <origin xyz="0 0 -${sphere_wheel_offset}" rpy="0 -0 0" />
       <geometry>
-        <mesh filename="package://catbot_description/meshes/collision/wheel_assm_3_collision.stl" />
+        <!-- <mesh filename="package://catbot_description/meshes/collision/wheel_assm_3_collision.stl" /> -->
+        <sphere radius="${wheel_radius}"/>
       </geometry>
     </collision>
@@ -149,5 +153,5 @@
   <link name="wheel_assm_4">
     <visual>
-      <origin xyz="0 0 0" rpy="0 -0 0" />
+      <origin xyz="0 0 ${sphere_wheel_offset}" rpy="0 -0 0" />
       <geometry>
         <mesh filename="package://catbot_description/meshes/visual/wheel_assm_4_visual.stl" />
@@ -160,5 +164,6 @@
       <origin xyz="0 0 0" rpy="0 -0 0" />
       <geometry>
-        <mesh filename="package://catbot_description/meshes/collision/wheel_assm_4_collision.stl" />
+        <!-- <mesh filename="package://catbot_description/meshes/collision/wheel_assm_4_collision.stl" /> -->
+        <sphere radius="${wheel_radius}"/>
       </geometry>
     </collision>

Commit message: align Gazebo and RViz correctly

File: src/catbot_description/urdf/catbot/catbot_macro.xacro (robot description, xacro)
@@ -7,5 +7,6 @@
     <parent link="base_link" />
     <child link="still_chassis_assm" />
-    <origin rpy="0.0 0 0" xyz="0 0 0" />
+    <!-- rotate 90deg to orient correctly -->
+    <origin rpy="0.0 0 1.5708" xyz="0 0 0" />
   </joint>
   <link name="still_chassis_assm">

Commit message: swap back to real wheel shapes

File: src/catbot_description/urdf/catbot/catbot_macro.xacro (robot description, xacro)
@@ -51,6 +51,6 @@
       <origin xyz="0 0 -${sphere_wheel_offset}" rpy="0 -0 0" />
       <geometry>
-        <!-- <mesh filename="package://catbot_description/meshes/collision/wheel_assm_collision.stl" /> -->
-        <sphere radius="${wheel_radius}"/>
+        <mesh filename="package://catbot_description/meshes/collision/wheel_assm_collision.stl" />
+        <!-- <sphere radius="${wheel_radius}"/> -->
       </geometry>
     </collision>
@@ -87,6 +87,6 @@
       <origin xyz="0 0 -${sphere_wheel_offset}" rpy="0 -0 0" />
       <geometry>
-        <!-- <mesh filename="package://catbot_description/meshes/collision/wheel_assm_2_collision.stl" /> -->
-        <sphere radius="${wheel_radius}"/>
+        <mesh filename="package://catbot_description/meshes/collision/wheel_assm_2_collision.stl" />
+        <!-- <sphere radius="${wheel_radius}"/> -->
       </geometry>
     </collision>
@@ -123,6 +123,6 @@
       <origin xyz="0 0 -${sphere_wheel_offset}" rpy="0 -0 0" />
       <geometry>
-        <!-- <mesh filename="package://catbot_description/meshes/collision/wheel_assm_3_collision.stl" /> -->
-        <sphere radius="${wheel_radius}"/>
+        <mesh filename="package://catbot_description/meshes/collision/wheel_assm_3_collision.stl" />
+        <!-- <sphere radius="${wheel_radius}"/> -->
       </geometry>
     </collision>
@@ -159,6 +159,6 @@
       <origin xyz="0 0 0" rpy="0 -0 0" />
       <geometry>
-        <!-- <mesh filename="package://catbot_description/meshes/collision/wheel_assm_4_collision.stl" /> -->
-        <sphere radius="${wheel_radius}"/>
+        <mesh filename="package://catbot_description/meshes/collision/wheel_assm_4_collision.stl" />
+        <!-- <sphere radius="${wheel_radius}"/> -->
       </geometry>
     </collision>

Commit message: removed leftover sphere wheel artifacts

File: src/catbot_description/urdf/catbot/catbot_macro.xacro (robot description, xacro)
@@ -49,8 +49,7 @@
     </visual>
     <collision>
-      <origin xyz="0 0 -${sphere_wheel_offset}" rpy="0 -0 0" />
+      <origin xyz="0 0 0" rpy="0 -0 0" />
       <geometry>
         <mesh filename="package://catbot_description/meshes/collision/wheel_assm_collision.stl" />
-        <!-- <sphere radius="${wheel_radius}"/> -->
       </geometry>
     </collision>
@@ -85,8 +84,7 @@
     </visual>
     <collision>
-      <origin xyz="0 0 -${sphere_wheel_offset}" rpy="0 -0 0" />
+      <origin xyz="0 0 0" rpy="0 -0 0" />
       <geometry>
         <mesh filename="package://catbot_description/meshes/collision/wheel_assm_2_collision.stl" />
-        <!-- <sphere radius="${wheel_radius}"/> -->
       </geometry>
     </collision>
@@ -121,8 +119,7 @@
     </visual>
     <collision>
-      <origin xyz="0 0 -${sphere_wheel_offset}" rpy="0 -0 0" />
+      <origin xyz="0 0 0" rpy="0 -0 0" />
       <geometry>
         <mesh filename="package://catbot_description/meshes/collision/wheel_assm_3_collision.stl" />
-        <!-- <sphere radius="${wheel_radius}"/> -->
       </geometry>
     </collision>
@@ -148,5 +145,5 @@
   <link name="wheel_assm_4">
     <visual>
-      <origin xyz="0 0 ${sphere_wheel_offset}" rpy="0 -0 0" />
+      <origin xyz="0 0 0" rpy="0 -0 0" />
       <geometry>
         <mesh filename="package://catbot_description/meshes/visual/wheel_assm_4_visual.stl" />
@@ -160,5 +157,4 @@
       <geometry>
         <mesh filename="package://catbot_description/meshes/collision/wheel_assm_4_collision.stl" />
-        <!-- <sphere radius="${wheel_radius}"/> -->
       </geometry>
     </collision>

Commit message: simplfied collision wheels

File: src/catbot_description/urdf/catbot/catbot_macro.xacro (robot description, xacro)
@@ -2,5 +2,8 @@
 <robot xmlns:xacro="http://wiki.ros.org/xacro">
   <xacro:include filename="inertial_macros.xacro"/>
-  <xacro:property name="sphere_wheel_offset" value="0.006"/>
+  <!-- simplify wheels to cylinders for collision -->
+  <xacro:arg name="cyl_wheels" default="true"/>
+  <xacro:property name="cyl_wheel_offset" value="-0.006"/>
+  <!-- <xacro:property name="simplified_wheel_collision" value="true"/> -->
   <link name="base_link"></link>
   <joint name="chassis_joint" type="fixed">
@@ -8,5 +11,5 @@
     <child link="still_chassis_assm" />
     <!-- rotate 90deg to orient correctly -->
-    <origin rpy="0.0 0 1.5708" xyz="0 0 0" />
+    <origin xyz="0 0 0" rpy="0.0 0 1.57" />
   </joint>
   <link name="still_chassis_assm">
@@ -49,8 +52,14 @@
     </visual>
     <collision>
-      <origin xyz="0 0 0" rpy="0 -0 0" />
-      <geometry>
-        <mesh filename="package://catbot_description/meshes/collision/wheel_assm_collision.stl" />
-      </geometry>
+      <xacro:if value="$(arg cyl_wheels)">
+        <origin xyz="0 0 ${cyl_wheel_offset}" rpy="0 -0 0" />
+        <xacro:wheel_cylinder_collision/>
+      </xacro:if>
+      <xacro:unless value="$(arg cyl_wheels)">
+        <origin xyz="0 0 0" rpy="0 -0 0" />
+        <geometry>
+          <mesh filename="package://catbot_description/meshes/collision/wheel_assm_collision.stl" />
+        </geometry>
+      </xacro:unless>
     </collision>
     <inertial>
@@ -72,4 +81,5 @@
     <child link="wheel_assm" />
     <axis xyz="0 0 1" />
+    <limit effort="1" velocity="20" />
   </joint>
   <link name="wheel_assm_2">
@@ -84,8 +94,14 @@
     </visual>
     <collision>
-      <origin xyz="0 0 0" rpy="0 -0 0" />
-      <geometry>
-        <mesh filename="package://catbot_description/meshes/collision/wheel_assm_2_collision.stl" />
-      </geometry>
+      <xacro:if value="$(arg cyl_wheels)">
+        <origin xyz="0 0 ${cyl_wheel_offset}" rpy="0 -0 0" />
+        <xacro:wheel_cylinder_collision/>
+      </xacro:if>
+      <xacro:unless value="$(arg cyl_wheels)">
+        <origin xyz="0 0 0" rpy="0 -0 0" />
+        <geometry>
+          <mesh filename="package://catbot_description/meshes/collision/wheel_assm_2_collision.stl" />
+        </geometry>
+      </xacro:unless>
     </collision>
     <inertial>
@@ -107,4 +123,5 @@
     <child link="wheel_assm_2" />
     <axis xyz="0 0 1" />
+    <limit effort="1" velocity="20" />
   </joint>
   <link name="wheel_assm_3">
@@ -119,8 +136,14 @@
     </visual>
     <collision>
-      <origin xyz="0 0 0" rpy="0 -0 0" />
-      <geometry>
-        <mesh filename="package://catbot_description/meshes/collision/wheel_assm_3_collision.stl" />
-      </geometry>
+      <xacro:if value="$(arg cyl_wheels)">
+        <origin xyz="0 0 ${cyl_wheel_offset}" rpy="0 -0 0" />
+        <xacro:wheel_cylinder_collision/>
+      </xacro:if>
+      <xacro:unless value="$(arg cyl_wheels)">
+        <origin xyz="0 0 0" rpy="0 -0 0" />
+        <geometry>
+          <mesh filename="package://catbot_description/meshes/collision/wheel_assm_3_collision.stl" />
+        </geometry>
+      </xacro:unless>
     </collision>
     <inertial>
@@ -142,4 +165,5 @@
     <child link="wheel_assm_3" />
     <axis xyz="0 0 1" />
+    <limit effort="1" velocity="20" />
   </joint>
   <link name="wheel_assm_4">
@@ -154,8 +178,14 @@
     </visual>
     <collision>
-      <origin xyz="0 0 0" rpy="0 -0 0" />
-      <geometry>
-        <mesh filename="package://catbot_description/meshes/collision/wheel_assm_4_collision.stl" />
-      </geometry>
+      <xacro:if value="$(arg cyl_wheels)">
+        <origin xyz="0 0 ${cyl_wheel_offset}" rpy="0 -0 0" />
+        <xacro:wheel_cylinder_collision/>
+      </xacro:if>
+      <xacro:unless value="$(arg cyl_wheels)">
+        <origin xyz="0 0 0" rpy="0 -0 0" />
+        <geometry>
+          <mesh filename="package://catbot_description/meshes/collision/wheel_assm_4_collision.stl" />
+        </geometry>
+      </xacro:unless>
     </collision>
     <inertial>
@@ -177,4 +207,5 @@
     <child link="wheel_assm_4" />
     <axis xyz="0 0 -1" />
+    <limit effort="1" velocity="20" />
   </joint>
 </robot>

File: src/catbot_description/urdf/catbot/inertial_macros.xacro (robot description, xacro)
@@ -49,3 +49,8 @@
         </xacro:inertial_box>
     </xacro:macro>
+    <xacro:macro name="wheel_cylinder_collision">
+        <geometry>
+            <cylinder length="${wheel_thickness}" radius="${wheel_radius}"/>
+        </geometry>
+    </xacro:macro>
 </robot>

File: src/catbot_description/urdf/gazebo_catbot.xacro (robot description, xacro)
@@ -1,4 +1,11 @@
 <?xml version="1.0" ?>
 <robot xmlns:xacro="http://ros.org/wiki/xacro">
+    <xacro:macro name="gz_wheel_physics">
+        <!-- <mu1 value="1.0"/>
+        <mu2 value="0.5"/>
+        <kp value="10000000.0"/>
+        <kd value="1.0"/> -->
+        <!-- <fdir1 value="1 0 0"/> -->
+    </xacro:macro>
     <gazebo reference="still_chassis_assm">
         <material>Gazebo/Green</material>
@@ -6,17 +13,17 @@
     <gazebo reference="wheel_assm">
         <material>Gazebo/Black</material>
-        <mu1 value="0.001"/>
-        <mu2 value="0.001"/>
+        <xacro:gz_wheel_physics/>
     </gazebo>
     <gazebo reference="wheel_assm_2">
         <material>Gazebo/Blue</material>
+        <xacro:gz_wheel_physics/>
     </gazebo>
     <gazebo reference="wheel_assm_3">
         <material>Gazebo/Black</material>
-        <mu1 value="0.001"/>
-        <mu2 value="0.001"/>
+        <xacro:gz_wheel_physics/>
     </gazebo>
     <gazebo reference="wheel_assm_4">
         <material>Gazebo/Blue</material>
+        <xacro:gz_wheel_physics/>
     </gazebo>
 </robot>
