Commit message: renamed wheel joints

File: src/catbot_description/urdf/4wd_control.xacro (robot description, xacro)
@@ -8,8 +8,8 @@
         <num_wheel_pairs>2</num_wheel_pairs>
         <!-- Wheel Information -->
-        <left_joint>fl_wheel</left_joint>
-        <right_joint>rf_wheel</right_joint>
-        <left_joint>rl_wheel</left_joint>
-        <right_joint>rr_wheel</right_joint>
+        <left_joint>front_left_wheel_joint</left_joint>
+        <right_joint>front_right_wheel_joint</right_joint>
+        <left_joint>rear_left_wheel_joint</left_joint>
+        <right_joint>rear_right_wheel_joint</right_joint>
         <wheel_separation>${wheel_separation}</wheel_separation>
         <wheel_separation>${wheel_separation}</wheel_separation>

File: src/catbot_description/urdf/catbot/catbot_macro.xacro (robot description, xacro)
@@ -67,5 +67,5 @@
       </inertial>
   </link>
-  <joint name="rr_wheel" type="continuous">
+  <joint name="rear_right_wheel_joint" type="continuous">
     <origin xyz="-0.077614131532514007983 0.080478921592024327269 -0.030500000000000013212"
     rpy="-1.570796326794896558 0.67540343776289657463 -1.5707963267948956698" />
@@ -103,5 +103,5 @@
     </inertial>
   </link>
-  <joint name="rf_wheel" type="continuous">
+  <joint name="front_right_wheel_joint" type="continuous">
     <origin xyz="-0.077614131532534658131 -0.068021078407976207081 -0.030499999999999957701"
     rpy="1.570796326794896558 5.0445758681405589749e-15 1.570796326794896336" />
@@ -139,5 +139,5 @@
     </inertial>
   </link>
-  <joint name="rl_wheel" type="continuous">
+  <joint name="rear_left_wheel_joint" type="continuous">
     <origin xyz="0.078385868467483257871 0.080478921592024507681 -0.030500000000000044437"
     rpy="-1.570796326794896558 -5.0445758681405660746e-15 1.5707963267948970021" />
@@ -175,5 +175,5 @@
     </inertial>
   </link>
-  <joint name="fl_wheel" type="continuous">
+  <joint name="front_left_wheel_joint" type="continuous">
     <origin xyz="0.078385868467507308077 -0.068021078407975985036 -0.030500000000000034028"
     rpy="-1.5707963267949118791 1.5703086100333234487 1.5707963267962468112" />
