Commit message: updated ros2_control urdf

File: src/catbot_description/urdf/catbot.urdf.xacro (robot description, xacro)
@@ -9,5 +9,5 @@
   <xacro:arg name="simulation_controllers" default="" />
   <xacro:include filename="$(find catbot_description)/urdf/catbot/catbot_macro.xacro"/>
-  <!-- <xacro:include filename="$(find catbot_description)/urdf/catbot/catbot_macro.ros2_control.xacro"/> -->
+  <xacro:include filename="$(find catbot_description)/urdf/catbot/catbot_macro.ros2_control.xacro"/>
   <!-- create link fixed to the "world" -->
   <link name="world" />
@@ -17,5 +17,5 @@
     <origin xyz="0 0 0" rpy="0 0 0" />          <!-- position robot in the world -->
   </xacro:catbot>
-  <!-- <xacro:catbot_ros2_control
+  <xacro:catbot_ros2_control
     name="catbot"
     prefix="$(arg prefix)"
@@ -24,4 +24,4 @@
     sim_gazebo_classic="$(arg sim_gazebo_classic)"
     sim_gazebo="$(arg sim_gazebo)"
-    simulation_controllers="$(arg simulation_controllers)" /> -->
+    simulation_controllers="$(arg simulation_controllers)" />
 </robot>

File: src/catbot_description/urdf/catbot/catbot_macro.ros2_control.xacro (robot description, xacro)
@@ -26,91 +26,36 @@
         </xacro:unless>
       </hardware>
-      <joint name="${prefix}joint1">
-        <command_interface name="position">     <!-- Add/Remove interfaces as needed -->
-          <param name="min">-1</param>
-          <param name="max">1</param>
+      <joint name="${prefix}rr_wheel">
+        <command_interface name="velocity">
+          <param name="min">-10</param>
+          <param name="max">10</param>
         </command_interface>
-        <state_interface name="position">
-          <param name="initial_value">0.0</param>
-        </state_interface>
+        <state_interface name="position"/>
         <state_interface name="velocity"/>
-        <state_interface name="acceleration"/>
       </joint>
       <joint name="${prefix}joint2">
-        <command_interface name="position">     <!-- Add/Remove interfaces as needed -->
-          <param name="min">-1</param>
-          <param name="max">1</param>
+        <command_interface name="velocity">
+          <param name="min">-10</param>
+          <param name="max">10</param>
         </command_interface>
-        <state_interface name="position">
-          <param name="initial_value">0.0</param>
-        </state_interface>
+        <state_interface name="position"/>
         <state_interface name="velocity"/>
-        <state_interface name="acceleration"/>
       </joint>
       <joint name="${prefix}joint3">
-        <command_interface name="position">     <!-- Add/Remove interfaces as needed -->
-          <param name="min">-1</param>
-          <param name="max">1</param>
+        <command_interface name="velocity">
+          <param name="min">-10</param>
+          <param name="max">10</param>
         </command_interface>
-        <state_interface name="position">
-          <param name="initial_value">0.0</param>
-        </state_interface>
+        <state_interface name="position"/>
         <state_interface name="velocity"/>
-        <state_interface name="acceleration"/>
       </joint>
       <joint name="${prefix}joint4">
-        <command_interface name="position">     <!-- Add/Remove interfaces as needed -->
-          <param name="min">-1</param>
-          <param name="max">1</param>
+        <command_interface name="velocity">
+          <param name="min">-10</param>
+          <param name="max">10</param>
         </command_interface>
-        <state_interface name="position">
-          <param name="initial_value">0.0</param>
-        </state_interface>
+        <state_interface name="position"/>
         <state_interface name="velocity"/>
-        <state_interface name="acceleration"/>
       </joint>
-      <joint name="${prefix}joint5">
-        <command_interface name="position">     <!-- Add/Remove interfaces as needed -->
-          <param name="min">-1</param>
-          <param name="max">1</param>
-        </command_interface>
-        <state_interface name="position">
-          <param name="initial_value">0.0</param>
-        </state_interface>
-        <state_interface name="velocity"/>
-        <state_interface name="acceleration"/>
-      </joint>
-      <joint name="${prefix}joint6">
-        <command_interface name="position">     <!-- Add/Remove interfaces as needed -->
-          <param name="min">-1</param>
-          <param name="max">1</param>
-        </command_interface>
-        <state_interface name="position">
-          <param name="initial_value">0.0</param>
-        </state_interface>
-        <state_interface name="velocity"/>
-        <state_interface name="acceleration"/>
-      </joint>
-      <sensor name="tcp_fts_sensor">            <!-- Remove/change sensors as needed -->
-        <state_interface name="fx"/>
-        <state_interface name="fy"/>
-        <state_interface name="fz"/>
-        <state_interface name="tx"/>
-        <state_interface name="ty"/>
-        <state_interface name="tz"/>
-        <param name="frame_id">tool0</param>    <!-- Change sensors as needed -->
-        <param name="min_fx">-100</param>
-        <param name="max_fx">100</param>
-        <param name="min_fy">-100</param>
-        <param name="max_fy">100</param>
-        <param name="min_fz">-200</param>
-        <param name="max_fz">200</param>
-        <param name="min_tx">-10</param>
-        <param name="max_tx">10</param>
-        <param name="min_ty">-10</param>
-        <param name="max_ty">10</param>
-        <param name="min_tz">-15</param>
-        <param name="max_tz">15</param>
-      </sensor>
     </ros2_control>
     <xacro:if value="$(arg sim_gazebo_classic)">

Commit message: take out of gazebo floor

File: src/catbot_description/urdf/catbot.urdf.xacro (robot description, xacro)
@@ -16,5 +16,5 @@
   <!-- set prefix if multiple robots are used -->
   <xacro:catbot prefix="$(arg prefix)" parent="world" >
-    <origin xyz="0 0 0" rpy="0 0 0" />          <!-- position robot in the world -->
+    <origin xyz="0 0 0.0635" rpy="0 0 0" />          <!-- position robot in the world -->
   </xacro:catbot>
   <xacro:catbot_ros2_control

Commit message: GRAVITY WORKSgit add src/catbot_description

File: src/catbot_description/urdf/catbot.urdf.xacro (robot description, xacro)
@@ -17,11 +17,6 @@
     <xacro:include filename="gazebo_control.xacro" />
   </xacro:unless>
-  <!-- create link fixed to the "world" -->
-  <link name="world" />
   <!-- Load robot's macro with parameters -->
   <!-- set prefix if multiple robots are used -->
-  <xacro:catbot prefix="$(arg prefix)" parent="world" >
-    <origin xyz="0 0 0.0635" rpy="0 0 0" />          <!-- position robot in the world -->
-  </xacro:catbot>
   <xacro:if value="$(arg use_ros2_control)">
     <xacro:catbot_ros2_control

File: src/catbot_description/urdf/catbot/catbot_macro.xacro (robot description, xacro)
@@ -1,144 +1,136 @@
 <?xml version="1.0" encoding="utf-8"?>
 <robot xmlns:xacro="http://wiki.ros.org/xacro">
-  <xacro:macro name="catbot" params="prefix parent *origin">
-    <xacro:include filename="inertial_macros.xacro"/>
-    <!-- base_joint fixes base_link to the environment -->
-    <joint name="${prefix}base_joint" type="fixed">
-      <xacro:insert_block name="origin" />
-      <parent link="${parent}" />
-      <child link="${prefix}base_link" />
-    </joint>
-    <link name="base_link"></link>
-    <joint name="base_link_to_base" type="fixed">
-      <parent link="base_link" />
-      <child link="still_chassis_assm" />
-      <origin rpy="0.0 0 0" xyz="0 0 0" />
-    </joint>
-    <link name="still_chassis_assm">
-      <visual>
-        <origin xyz="0 0 0" rpy="0 -0 0" />
-        <geometry>
-          <mesh filename="package://catbot_description/meshes/visual/still_chassis_assm_visual.stl" />
-        </geometry>
-        <material name="still_chassis_assm_material">
-          <color rgba="0.66987717125153911635 0.81712318213796708566 0.66602980483018847657 1.0" />
-        </material>
-      </visual>
-      <collision>
-        <origin xyz="0 0 0" rpy="0 -0 0" />
-        <geometry>
-          <mesh filename="package://catbot_description/meshes/collision/still_chassis_assm_collision.stl" />
-        </geometry>
-      </collision>
-      <xacro:chassis_inertia/>
-    </link>
-    <link name="wheel_assm">
-      <visual>
-        <origin xyz="0 0 0" rpy="0 -0 0" />
-        <geometry>
-          <mesh filename="package://catbot_description/meshes/visual/wheel_assm_visual.stl" />
-        </geometry>
-        <material name="wheel_assm_material">
-          <color rgba="0.34876043041436377568 0.28454440741211711741 0.12249285133838178075 1.0" />
-        </material>
-      </visual>
-      <collision>
-        <origin xyz="0 0 0" rpy="0 -0 0" />
-        <geometry>
-          <mesh filename="package://catbot_description/meshes/collision/wheel_assm_collision.stl" />
-        </geometry>
-      </collision>
-      <xacro:wheel_inertia/>
-    </link>
-    <joint name="rr_wheel" type="continuous">
-      <origin xyz="-0.077614131532514007983 0.080478921592024327269 -0.030500000000000013212"
-      rpy="-1.570796326794896558 0.67540343776289657463 -1.5707963267948956698" />
-      <parent link="still_chassis_assm" />
-      <child link="wheel_assm" />
-      <axis xyz="0 0 1" />
-      <limit effort="1" velocity="20" />
-      <joint_properties friction="0.0" />
-    </joint>
-    <link name="wheel_assm_2">
-      <visual>
-        <origin xyz="0 0 0" rpy="0 -0 0" />
-        <geometry>
-          <mesh filename="package://catbot_description/meshes/visual/wheel_assm_2_visual.stl" />
-        </geometry>
-        <material name="wheel_assm_2_material">
-          <color rgba="0.34876043041436377568 0.28454440741211711741 0.12249285133838178075 1.0" />
-        </material>
-      </visual>
-      <collision>
-        <origin xyz="0 0 0" rpy="0 -0 0" />
-        <geometry>
-          <mesh filename="package://catbot_description/meshes/collision/wheel_assm_2_collision.stl" />
-        </geometry>
-      </collision>
-      <xacro:wheel_inertia/>
-    </link>
-    <joint name="rf_wheel" type="continuous">
-      <origin xyz="-0.077614131532534658131 -0.068021078407976207081 -0.030499999999999957701"
-      rpy="1.570796326794896558 5.0445758681405589749e-15 1.570796326794896336" />
-      <parent link="still_chassis_assm" />
-      <child link="wheel_assm_2" />
-      <axis xyz="0 0 1" />
-      <limit effort="1" velocity="20" />
-      <joint_properties friction="0.0" />
-    </joint>
-    <link name="wheel_assm_3">
-      <visual>
-        <origin xyz="0 0 0" rpy="0 -0 0" />
-        <geometry>
-          <mesh filename="package://catbot_description/meshes/visual/wheel_assm_3_visual.stl" />
-        </geometry>
-        <material name="wheel_assm_3_material">
-          <color rgba="0.34876043041436383119 0.28454440741211711741 0.12249285133838178075 1.0" />
-        </material>
-      </visual>
-      <collision>
-        <origin xyz="0 0 0" rpy="0 -0 0" />
-        <geometry>
-          <mesh filename="package://catbot_description/meshes/collision/wheel_assm_3_collision.stl" />
-        </geometry>
-      </collision>
-      <xacro:wheel_inertia/>
-    </link>
-    <joint name="rl_wheel" type="continuous">
-      <origin xyz="0.078385868467483257871 0.080478921592024507681 -0.030500000000000044437"
-      rpy="-1.570796326794896558 -5.0445758681405660746e-15 1.5707963267948970021" />
-      <parent link="still_chassis_assm" />
-      <child link="wheel_assm_3" />
-      <axis xyz="0 0 1" />
-      <limit effort="1" velocity="20" />
-      <joint_properties friction="0.0" />
-    </joint>
-    <link name="wheel_assm_4">
-      <visual>
-        <origin xyz="0 0 0" rpy="0 -0 0" />
-        <geometry>
-          <mesh filename="package://catbot_description/meshes/visual/wheel_assm_4_visual.stl" />
-        </geometry>
-        <material name="wheel_assm_4_material">
-          <color rgba="0.34876043041436377568 0.28454440741211711741 0.12249285133838176687 1.0" />
-        </material>
-      </visual>
-      <collision>
-        <origin xyz="0 0 0" rpy="0 -0 0" />
-        <geometry>
-          <mesh filename="package://catbot_description/meshes/collision/wheel_assm_4_collision.stl" />
-        </geometry>
-      </collision>
-      <xacro:wheel_inertia/>
-    </link>
-    <joint name="fl_wheel" type="continuous">
-      <origin xyz="0.078385868467507308077 -0.068021078407975985036 -0.030500000000000034028"
-      rpy="-1.5707963267949118791 1.5703086100333234487 1.5707963267962468112" />
-      <parent link="still_chassis_assm" />
-      <child link="wheel_assm_4" />
-      <axis xyz="0 0 1" />
-      <limit effort="1" velocity="20" />
-      <joint_properties friction="0.0" />
-    </joint>
-  </xacro:macro>
+  <xacro:include filename="inertial_macros.xacro"/>
+  <link name="base_link"></link>
+  <joint name="chassis_joint" type="fixed">
+    <parent link="base_link" />
+    <child link="still_chassis_assm" />
+    <origin rpy="0.0 0 0" xyz="0 0 0" />
+  </joint>
+  <link name="still_chassis_assm">
+    <visual>
+      <origin xyz="0 0 0" rpy="0 -0 0" />
+      <geometry>
+        <mesh filename="package://catbot_description/meshes/visual/still_chassis_assm_visual.stl" />
+      </geometry>
+      <material name="still_chassis_assm_material">
+        <color rgba="0.66987717125153911635 0.81712318213796708566 0.66602980483018847657 1.0" />
+      </material>
+    </visual>
+    <collision>
+      <origin xyz="0 0 0" rpy="0 -0 0" />
+      <geometry>
+        <mesh filename="package://catbot_description/meshes/collision/still_chassis_assm_collision.stl" />
+      </geometry>
+    </collision>
+    <xacro:chassis_inertia/>
+  </link>
+  <link name="wheel_assm">
+    <visual>
+      <origin xyz="0 0 0" rpy="0 -0 0" />
+      <geometry>
+        <mesh filename="package://catbot_description/meshes/visual/wheel_assm_visual.stl" />
+      </geometry>
+      <material name="wheel_assm_material">
+        <color rgba="0.34876043041436377568 0.28454440741211711741 0.12249285133838178075 1.0" />
+      </material>
+    </visual>
+    <collision>
+      <origin xyz="0 0 0" rpy="0 -0 0" />
+      <geometry>
+        <mesh filename="package://catbot_description/meshes/collision/wheel_assm_collision.stl" />
+      </geometry>
+    </collision>
+    <xacro:wheel_inertia/>
+  </link>
+  <joint name="rr_wheel" type="continuous">
+    <origin xyz="-0.077614131532514007983 0.080478921592024327269 -0.030500000000000013212"
+    rpy="-1.570796326794896558 0.67540343776289657463 -1.5707963267948956698" />
+    <parent link="still_chassis_assm" />
+    <child link="wheel_assm" />
+    <axis xyz="0 0 1" />
+    <limit effort="1" velocity="20" />
+    <joint_properties friction="0.0" />
+  </joint>
+  <link name="wheel_assm_2">
+    <visual>
+      <origin xyz="0 0 0" rpy="0 -0 0" />
+      <geometry>
+        <mesh filename="package://catbot_description/meshes/visual/wheel_assm_2_visual.stl" />
+      </geometry>
+      <material name="wheel_assm_2_material">
+        <color rgba="0.34876043041436377568 0.28454440741211711741 0.12249285133838178075 1.0" />
+      </material>
+    </visual>
+    <collision>
+      <origin xyz="0 0 0" rpy="0 -0 0" />
+      <geometry>
+        <mesh filename="package://catbot_description/meshes/collision/wheel_assm_2_collision.stl" />
+      </geometry>
+    </collision>
+    <xacro:wheel_inertia/>
+  </link>
+  <joint name="rf_wheel" type="continuous">
+    <origin xyz="-0.077614131532534658131 -0.068021078407976207081 -0.030499999999999957701"
+    rpy="1.570796326794896558 5.0445758681405589749e-15 1.570796326794896336" />
+    <parent link="still_chassis_assm" />
+    <child link="wheel_assm_2" />
+    <axis xyz="0 0 1" />
+    <limit effort="1" velocity="20" />
+    <joint_properties friction="0.0" />
+  </joint>
+  <link name="wheel_assm_3">
+    <visual>
+      <origin xyz="0 0 0" rpy="0 -0 0" />
+      <geometry>
+        <mesh filename="package://catbot_description/meshes/visual/wheel_assm_3_visual.stl" />
+      </geometry>
+      <material name="wheel_assm_3_material">
+        <color rgba="0.34876043041436383119 0.28454440741211711741 0.12249285133838178075 1.0" />
+      </material>
+    </visual>
+    <collision>
+      <origin xyz="0 0 0" rpy="0 -0 0" />
+      <geometry>
+        <mesh filename="package://catbot_description/meshes/collision/wheel_assm_3_collision.stl" />
+      </geometry>
+    </collision>
+    <xacro:wheel_inertia/>
+  </link>
+  <joint name="rl_wheel" type="continuous">
+    <origin xyz="0.078385868467483257871 0.080478921592024507681 -0.030500000000000044437"
+    rpy="-1.570796326794896558 -5.0445758681405660746e-15 1.5707963267948970021" />
+    <parent link="still_chassis_assm" />
+    <child link="wheel_assm_3" />
+    <axis xyz="0 0 1" />
+    <limit effort="1" velocity="20" />
+    <joint_properties friction="0.0" />
+  </joint>
+  <link name="wheel_assm_4">
+    <visual>
+      <origin xyz="0 0 0" rpy="0 -0 0" />
+      <geometry>
+        <mesh filename="package://catbot_description/meshes/visual/wheel_assm_4_visual.stl" />
+      </geometry>
+      <material name="wheel_assm_4_material">
+        <color rgba="0.34876043041436377568 0.28454440741211711741 0.12249285133838176687 1.0" />
+      </material>
+    </visual>
+    <collision>
+      <origin xyz="0 0 0" rpy="0 -0 0" />
+      <geometry>
+        <mesh filename="package://catbot_description/meshes/collision/wheel_assm_4_collision.stl" />
+      </geometry>
+    </collision>
+    <xacro:wheel_inertia/>
+  </link>
+  <joint name="fl_wheel" type="continuous">
+    <origin xyz="0.078385868467507308077 -0.068021078407975985036 -0.030500000000000034028"
+    rpy="-1.5707963267949118791 1.5703086100333234487 1.5707963267962468112" />
+    <parent link="still_chassis_assm" />
+    <child link="wheel_assm_4" />
+    <axis xyz="0 0 1" />
+    <limit effort="1" velocity="20" />
+    <joint_properties friction="0.0" />
+  </joint>
 </robot>
