Commit message: Feature/gazebo (#23)
* updated ros2_control urdf

* package genreated by RTW

* made pre-commit global

* Fixed invisible gazebo model by exporting in package.xml
``` <export>
        <gazebo_ros gazebo_model_path="${prefix}/.." />
    </export>
```

* color for gazebo

* python intellisense update

* remove annoying spellcheck

* articulated robotics-based Robot State publisher 

* config for gazebo plugin accurate for catbot

* update from onshape again

* swapped to fixed rear wheels for testing

* works FWD!

* update README

* added inline formatting ignore commands

File: src/catbot_description/urdf/catbot.urdf.xacro (robot description, xacro)
@@ -3,4 +3,5 @@
   <!-- Use this if parameters are set from the launch file, otherwise delete -->
   <xacro:arg name="prefix" default="" />
+  <xacro:arg name="use_ros2_control" default="false"/>
   <xacro:arg name="use_mock_hardware" default="false" />
   <xacro:arg name="mock_sensor_commands" default="false" />
@@ -9,19 +10,22 @@
   <xacro:arg name="simulation_controllers" default="" />
   <xacro:include filename="$(find catbot_description)/urdf/catbot/catbot_macro.xacro"/>
-  <!-- <xacro:include filename="$(find catbot_description)/urdf/catbot/catbot_macro.ros2_control.xacro"/> -->
-  <!-- create link fixed to the "world" -->
-  <link name="world" />
+  <xacro:include filename="gazebo_catbot.xacro" />
+  <xacro:if value="$(arg use_ros2_control)">
+    <xacro:include filename="$(find catbot_description)/urdf/catbot/catbot_macro.ros2_control.xacro"/>
+  </xacro:if>
+  <xacro:unless value="$(arg use_ros2_control)">
+    <xacro:include filename="gazebo_control.xacro" />
+  </xacro:unless>
   <!-- Load robot's macro with parameters -->
   <!-- set prefix if multiple robots are used -->
-  <xacro:catbot prefix="$(arg prefix)" parent="world" >
-    <origin xyz="0 0 0" rpy="0 0 0" />          <!-- position robot in the world -->
-  </xacro:catbot>
-  <!-- <xacro:catbot_ros2_control
-    name="catbot"
-    prefix="$(arg prefix)"
-    use_mock_hardware="$(arg use_mock_hardware)"
-    mock_sensor_commands="$(arg mock_sensor_commands)"
-    sim_gazebo_classic="$(arg sim_gazebo_classic)"
-    sim_gazebo="$(arg sim_gazebo)"
-    simulation_controllers="$(arg simulation_controllers)" /> -->
+  <xacro:if value="$(arg use_ros2_control)">
+    <xacro:catbot_ros2_control
+      name="catbot"
+      prefix="$(arg prefix)"
+      use_mock_hardware="$(arg use_mock_hardware)"
+      mock_sensor_commands="$(arg mock_sensor_commands)"
+      sim_gazebo_classic="$(arg sim_gazebo_classic)"
+      sim_gazebo="$(arg sim_gazebo)"
+      simulation_controllers="$(arg simulation_controllers)" />
+  </xacro:if>
 </robot>

File: src/catbot_description/urdf/catbot/catbot_macro.xacro (robot description, xacro)
@@ -1,193 +1,186 @@
 <?xml version="1.0" encoding="utf-8"?>
 <robot xmlns:xacro="http://wiki.ros.org/xacro">
-  <xacro:macro name="catbot" params="prefix parent *origin">
-    <!-- base_joint fixes base_link to the environment -->
-    <joint name="${prefix}base_joint" type="fixed">
-      <xacro:insert_block name="origin" />
-      <parent link="${parent}" />
-      <child link="${prefix}base_link" />
-    </joint>
-    <link name="base_link"></link>
-    <joint name="base_link_to_base" type="fixed">
-      <parent link="base_link" />
-      <child link="still_chassis_assm" />
-      <origin rpy="0.0 0 0" xyz="0 0 0" />
-    </joint>
-    <link name="still_chassis_assm">
-      <visual>
-        <origin xyz="0 0 0" rpy="0 -0 0" />
-        <geometry>
-          <mesh filename="package://catbot_description/meshes/visual/still_chassis_assm_visual.stl" />
-        </geometry>
-        <material name="still_chassis_assm_material">
-          <color rgba="0.66987717125153900533 0.81712318213796708566 0.66602980483018836555 1.0" />
-        </material>
-      </visual>
-      <collision>
-        <origin xyz="0 0 0" rpy="0 -0 0" />
-        <geometry>
-          <mesh filename="package://catbot_description/meshes/collision/still_chassis_assm_collision.stl" />
-        </geometry>
-      </collision>
-      <inertial>
-        <origin xyz="0.00027961412402240977014 0.0046876789374875839009 -0.0054409557585405705568"
+  <xacro:include filename="inertial_macros.xacro"/>
+  <link name="base_link"></link>
+  <joint name="chassis_joint" type="fixed">
+    <parent link="base_link" />
+    <child link="still_chassis_assm" />
+    <origin rpy="0.0 0 0" xyz="0 0 0" />
+  </joint>
+  <link name="still_chassis_assm">
+    <visual>
+      <origin xyz="0 0 0" rpy="0 -0 0" />
+      <geometry>
+        <mesh filename="package://catbot_description/meshes/visual/still_chassis_assm_visual.stl" />
+      </geometry>
+      <material name="still_chassis_assm_material">
+        <color rgba="0.66987717125153911635 0.81712318213796708566 0.66602980483018847657 1.0" />
+      </material>
+    </visual>
+    <collision>
+      <origin xyz="0 0 0" rpy="0 -0 0" />
+      <geometry>
+        <mesh filename="package://catbot_description/meshes/collision/still_chassis_assm_collision.stl" />
+      </geometry>
+    </collision>
+     <inertial>
+        <origin xyz="0.00027961412402240787278 0.0046876789374875821662 -0.0054409557585405705568"
         rpy="0 0 0" />
-        <mass value="1.0156681416365394011" />
+        <mass value="1.015668141636539179" />
         <inertia ixx="0.0065127126032337098738"
-        ixy="1.5566438777542365468e-07"
-        ixz="3.6708728527239328719e-06"
+        ixy="1.5566438777546685336e-07"
+        ixz="3.6708728527239311778e-06"
         iyy="0.0025991819436423468752"
-        iyz="6.1954470337197489749e-05"
+        iyz="6.1954470337197611722e-05"
         izz="0.0071648278899316356766" />
       </inertial>
-    </link>
-    <link name="wheel_assm">
-      <visual>
-        <origin xyz="0 0 0" rpy="0 -0 0" />
-        <geometry>
-          <mesh filename="package://catbot_description/meshes/visual/wheel_assm_visual.stl" />
-        </geometry>
-        <material name="wheel_assm_material">
-          <color rgba="0.34876043041436377568 0.28454440741211711741 0.12249285133838178075 1.0" />
-        </material>
-      </visual>
-      <collision>
-        <origin xyz="0 0 0" rpy="0 -0 0" />
-        <geometry>
-          <mesh filename="package://catbot_description/meshes/collision/wheel_assm_collision.stl" />
-        </geometry>
-      </collision>
-      <inertial>
-        <origin xyz="2.5876683231912983522e-09 -2.5321947387836322962e-09 -0.0043217676979120578026"
-        rpy="0 0 0" />
-        <mass value="0.054377782220193432439" />
-        <inertia ixx="1.7947780629583350172e-05"
-        ixy="-3.8234084814183779999e-12"
-        ixz="-1.6934852918263056535e-12"
-        iyy="1.7621269066491265109e-05"
-        iyz="-2.0136050751311128972e-12"
-        izz="2.8213568549230894094e-05" />
+  </link>
+  <link name="wheel_assm">
+    <visual>
+      <origin xyz="0 0 0" rpy="0 -0 0" />
+      <geometry>
+        <mesh filename="package://catbot_description/meshes/visual/wheel_assm_visual.stl" />
+      </geometry>
+      <material name="wheel_assm_material">
+        <color rgba="0.34876043041436377568 0.28454440741211711741 0.12249285133838178075 1.0" />
+      </material>
+    </visual>
+    <collision>
+      <origin xyz="0 0 0" rpy="0 -0 0" />
+      <geometry>
+        <mesh filename="package://catbot_description/meshes/collision/wheel_assm_collision.stl" />
+      </geometry>
+    </collision>
+    <inertial>
+      <origin xyz="2.5876683183573441879e-09 -2.5321947361304500679e-09 -0.0043217676979120569353"
+      rpy="0 0 0" />
+      <mass value="0.054377782220193432439" />
+      <inertia ixx="1.7947780629583346784e-05"
+      ixy="-3.8234084819748992999e-12"
+      ixz="-1.6934852924892931359e-12"
+      iyy="1.7621269066491268497e-05"
+      iyz="-2.0136050748759971485e-12"
+      izz="2.8213568549230894094e-05" />
       </inertial>
-    </link>
-    <joint name="rr_wheel" type="continuous">
-      <origin xyz="-0.077614131532514007983 0.080478921592024327269 -0.030500000000000013212"
-      rpy="-1.570796326794896558 0.67540343776289657463 -1.5707963267948956698" />
-      <parent link="still_chassis_assm" />
-      <child link="wheel_assm" />
-      <axis xyz="0 0 1" />
-      <limit effort="1" velocity="20" />
-      <joint_properties friction="0.0" />
-    </joint>
-    <link name="wheel_assm_2">
-      <visual>
-        <origin xyz="0 0 0" rpy="0 -0 0" />
-        <geometry>
-          <mesh filename="package://catbot_description/meshes/visual/wheel_assm_2_visual.stl" />
-        </geometry>
-        <material name="wheel_assm_2_material">
-          <color rgba="0.34876043041436377568 0.28454440741211711741 0.12249285133838178075 1.0" />
-        </material>
-      </visual>
-      <collision>
-        <origin xyz="0 0 0" rpy="0 -0 0" />
-        <geometry>
-          <mesh filename="package://catbot_description/meshes/collision/wheel_assm_2_collision.stl" />
-        </geometry>
-      </collision>
-      <inertial>
-        <origin xyz="2.5876683436570912888e-09 -2.5321947882875150234e-09 -0.0043217676979120907624"
-        rpy="0 0 0" />
-        <mass value="0.054377782220193432439" />
-        <inertia ixx="1.7947780629583373889e-05"
-        ixy="-3.8234084806256659389e-12"
-        ixz="-1.6934852952780513878e-12"
-        iyy="1.7621269066491271885e-05"
-        iyz="-2.0136050702142612672e-12"
-        izz="2.8213568549230904259e-05" />
-      </inertial>
-    </link>
-    <joint name="rf_wheel" type="continuous">
-      <origin xyz="-0.077614131532534658131 -0.068021078407976207081 -0.030499999999999957701"
-      rpy="1.570796326794896558 5.0445758681405589749e-15 1.570796326794896336" />
-      <parent link="still_chassis_assm" />
-      <child link="wheel_assm_2" />
-      <axis xyz="0 0 1" />
-      <limit effort="1" velocity="20" />
-      <joint_properties friction="0.0" />
-    </joint>
-    <link name="wheel_assm_3">
-      <visual>
-        <origin xyz="0 0 0" rpy="0 -0 0" />
-        <geometry>
-          <mesh filename="package://catbot_description/meshes/visual/wheel_assm_3_visual.stl" />
-        </geometry>
-        <material name="wheel_assm_3_material">
-          <color rgba="0.34876043041436383119 0.28454440741211711741 0.12249285133838178075 1.0" />
-        </material>
-      </visual>
-      <collision>
-        <origin xyz="0 0 0" rpy="0 -0 0" />
-        <geometry>
-          <mesh filename="package://catbot_description/meshes/collision/wheel_assm_3_collision.stl" />
-        </geometry>
-      </collision>
-      <inertial>
-        <origin xyz="2.5876683542375088732e-09 -2.5321947930490429075e-09 -0.0043217676979121003034"
-        rpy="0 0 0" />
-        <mass value="0.054377782220193432439" />
-        <inertia ixx="1.7947780629583373889e-05"
-        ixy="-3.8234084806256627077e-12"
-        ixz="-1.6934852942781941971e-12"
-        iyy="1.7621269066491275274e-05"
-        iyz="-2.01360506846477306e-12"
-        izz="2.8213568549230904259e-05" />
-      </inertial>
-    </link>
-    <joint name="rl_wheel" type="continuous">
-      <origin xyz="0.078385868467483257871 0.080478921592024507681 -0.030500000000000044437"
-      rpy="-1.570796326794896558 -5.0445758681405660746e-15 1.5707963267948970021" />
-      <parent link="still_chassis_assm" />
-      <child link="wheel_assm_3" />
-      <axis xyz="0 0 1" />
-      <limit effort="1" velocity="20" />
-      <joint_properties friction="0.0" />
-    </joint>
-    <link name="wheel_assm_4">
-      <visual>
-        <origin xyz="0 0 0" rpy="0 -0 0" />
-        <geometry>
-          <mesh filename="package://catbot_description/meshes/visual/wheel_assm_4_visual.stl" />
-        </geometry>
-        <material name="wheel_assm_4_material">
-          <color rgba="0.34876043041436377568 0.28454440741211711741 0.12249285133838176687 1.0" />
-        </material>
-      </visual>
-      <collision>
-        <origin xyz="0 0 0" rpy="0 -0 0" />
-        <geometry>
-          <mesh filename="package://catbot_description/meshes/collision/wheel_assm_4_collision.stl" />
-        </geometry>
-      </collision>
-      <inertial>
-        <origin xyz="2.5876682744584021363e-09 -2.5321945349340081079e-09 -0.0043217676979121323957"
-        rpy="0 0 0" />
-        <mass value="0.054377782220193432439" />
-        <inertia ixx="1.7947780629583377277e-05"
-        ixy="-3.8234084820191074185e-12"
-        ixz="-1.6934852985237760372e-12"
-        iyy="1.7621269066491275274e-05"
-        iyz="-2.0136050684267663727e-12"
-        izz="2.8213568549230907647e-05" />
-      </inertial>
-    </link>
-    <joint name="fl_wheel" type="continuous">
-      <origin xyz="0.078385868467507308077 -0.068021078407975985036 -0.030500000000000034028"
-      rpy="-1.5707963267949118791 1.5703086100333234487 1.5707963267962468112" />
-      <parent link="still_chassis_assm" />
-      <child link="wheel_assm_4" />
-      <axis xyz="0 0 1" />
-      <limit effort="1" velocity="20" />
-      <joint_properties friction="0.0" />
-    </joint>
-  </xacro:macro>
+  </link>
+  <joint name="rr_wheel" type="fixed">
+    <origin xyz="-0.077614131532514007983 0.080478921592024327269 -0.030500000000000013212"
+    rpy="-1.570796326794896558 0.67540343776289657463 -1.5707963267948956698" />
+    <parent link="still_chassis_assm" />
+    <child link="wheel_assm" />
+    <axis xyz="0 0 1" />
+    <!-- <limit effort="1" velocity="20" />
+    <joint_properties friction="0.0" /> -->
+  </joint>
+  <link name="wheel_assm_2">
+    <visual>
+      <origin xyz="0 0 0" rpy="0 -0 0" />
+      <geometry>
+        <mesh filename="package://catbot_description/meshes/visual/wheel_assm_2_visual.stl" />
+      </geometry>
+      <material name="wheel_assm_2_material">
+        <color rgba="0.34876043041436377568 0.28454440741211711741 0.12249285133838178075 1.0" />
+      </material>
+    </visual>
+    <collision>
+      <origin xyz="0 0 0" rpy="0 -0 0" />
+      <geometry>
+        <mesh filename="package://catbot_description/meshes/collision/wheel_assm_2_collision.stl" />
+      </geometry>
+    </collision>
+    <inertial>
+      <origin xyz="2.5876683388231371246e-09 -2.5321947856343332086e-09 -0.004321767697912089895"
+      rpy="0 0 0" />
+      <mass value="0.054377782220193432439" />
+      <inertia ixx="1.7947780629583370501e-05"
+      ixy="-3.8234084811821872389e-12"
+      ixz="-1.6934852959410392741e-12"
+      iyy="1.7621269066491275274e-05"
+      iyz="-2.013605069932675335e-12"
+      izz="2.8213568549230904259e-05" />
+    </inertial>
+  </link>
+  <joint name="rf_wheel" type="continuous">
+    <origin xyz="-0.077614131532534658131 -0.068021078407976207081 -0.030499999999999957701"
+    rpy="1.570796326794896558 5.0445758681405589749e-15 1.570796326794896336" />
+    <parent link="still_chassis_assm" />
+    <child link="wheel_assm_2" />
+    <axis xyz="0 0 1" />
+    <limit effort="1" velocity="20" />
+    <joint_properties friction="0.0" />
+  </joint>
+  <link name="wheel_assm_3">
+    <visual>
+      <origin xyz="0 0 0" rpy="0 -0 0" />
+      <geometry>
+        <mesh filename="package://catbot_description/meshes/visual/wheel_assm_3_visual.stl" />
+      </geometry>
+      <material name="wheel_assm_3_material">
+        <color rgba="0.34876043041436383119 0.28454440741211711741 0.12249285133838178075 1.0" />
+      </material>
+    </visual>
+    <collision>
+      <origin xyz="0 0 0" rpy="0 -0 0" />
+      <geometry>
+        <mesh filename="package://catbot_description/meshes/collision/wheel_assm_3_collision.stl" />
+      </geometry>
+    </collision>
+    <inertial>
+      <origin xyz="2.5876683494035538817e-09 -2.5321947903698363363e-09 -0.0043217676979121003034"
+      rpy="0 0 0" />
+      <mass value="0.054377782220193432439" />
+      <inertia ixx="1.7947780629583370501e-05"
+      ixy="-3.8234084811821831999e-12"
+      ixz="-1.6934852949411820834e-12"
+      iyy="1.7621269066491278662e-05"
+      iyz="-2.0136050682372531551e-12"
+      izz="2.8213568549230904259e-05" />
+    </inertial>
+  </link>
+  <joint name="rl_wheel" type="fixed">
+    <origin xyz="0.078385868467483257871 0.080478921592024507681 -0.030500000000000044437"
+    rpy="-1.570796326794896558 -5.0445758681405660746e-15 1.5707963267948970021" />
+    <parent link="still_chassis_assm" />
+    <child link="wheel_assm_3" />
+    <axis xyz="0 0 1" />
+    <!-- <limit effort="1" velocity="20" />
+    <joint_properties friction="0.0" /> -->
+  </joint>
+  <link name="wheel_assm_4">
+    <visual>
+      <origin xyz="0 0 0" rpy="0 -0 0" />
+      <geometry>
+        <mesh filename="package://catbot_description/meshes/visual/wheel_assm_4_visual.stl" />
+      </geometry>
+      <material name="wheel_assm_4_material">
+        <color rgba="0.34876043041436377568 0.28454440741211711741 0.12249285133838176687 1.0" />
+      </material>
+    </visual>
+    <collision>
+      <origin xyz="0 0 0" rpy="0 -0 0" />
+      <geometry>
+        <mesh filename="package://catbot_description/meshes/collision/wheel_assm_4_collision.stl" />
+      </geometry>
+    </collision>
+    <inertial>
+      <origin xyz="2.587668269624447972e-09 -2.5321945322547953329e-09 -0.0043217676979121323957"
+      rpy="0 0 0" />
+      <mass value="0.054377782220193432439" />
+      <inertia ixx="1.7947780629583373889e-05"
+      ixy="-3.8234084825756295263e-12"
+      ixz="-1.6934852991867637216e-12"
+      iyy="1.7621269066491278662e-05"
+      iyz="-2.0136050681091290175e-12"
+      izz="2.8213568549230907647e-05" />
+    </inertial>
+  </link>
+  <joint name="fl_wheel" type="continuous">
+    <origin xyz="0.078385868467507308077 -0.068021078407975985036 -0.030500000000000034028"
+    rpy="-1.5707963267949118791 1.5703086100333234487 1.5707963267962468112" />
+    <parent link="still_chassis_assm" />
+    <child link="wheel_assm_4" />
+    <axis xyz="0 0 -1" />
+    <limit effort="1" velocity="20" />
+    <joint_properties friction="0.0" />
+  </joint>
 </robot>
