Commit message: broken start of  integrate ros2 control.

File: src/catbot_description/urdf/catbot.urdf.xacro (robot description, xacro)
@@ -3,10 +3,6 @@
   <!-- Use this if parameters are set from the launch file, otherwise delete -->
   <xacro:arg name="prefix" default="" />
-  <xacro:arg name="use_ros2_control" default="false"/>
-  <xacro:arg name="use_mock_hardware" default="false" />
-  <xacro:arg name="mock_sensor_commands" default="false" />
-  <xacro:arg name="sim_gazebo_classic" default="false" />
-  <xacro:arg name="sim_gazebo" default="false" />
-  <xacro:arg name="simulation_controllers" default="" />
+  <xacro:arg name="use_ros2_control" default="true"/>
+  <xacro:arg name="sim_mode" default="false"/>
   <xacro:include filename="$(find catbot_description)/urdf/catbot/catbot_macro.xacro"/>
   <xacro:include filename="gazebo_catbot.xacro" />
@@ -19,6 +15,6 @@
   <!-- Load robot's macro with parameters -->
   <!-- set prefix if multiple robots are used -->
-  <xacro:if value="$(arg use_ros2_control)">
-    <xacro:catbot_ros2_control
+  <!-- <xacro:if value="$(arg use_ros2_control)"> -->
+    <!-- <xacro:catbot_ros2_control
       name="catbot"
       prefix="$(arg prefix)"
@@ -27,5 +23,5 @@
       sim_gazebo_classic="$(arg sim_gazebo_classic)"
       sim_gazebo="$(arg sim_gazebo)"
-      simulation_controllers="$(arg simulation_controllers)" />
-  </xacro:if>
+      simulation_controllers="$(arg simulation_controllers)" /> -->
+  <!-- </xacro:if>  -->
 </robot>

File: src/catbot_description/urdf/catbot/catbot_macro.ros2_control.xacro (robot description, xacro)
@@ -1,83 +1,47 @@
 <?xml version="1.0" encoding="UTF-8"?>
 <robot xmlns:xacro="http://wiki.ros.org/xacro">
-  <xacro:macro name="catbot_ros2_control" params="
-               name
-               prefix
-               use_mock_hardware:=^|false
-               mock_sensor_commands:=^|false
-               sim_gazebo_classic:=^|false
-               sim_gazebo:=^|false
-               simulation_controllers"
-               >
-    <ros2_control name="${name}" type="system">
-      <hardware>
-        <xacro:if value="${use_mock_hardware}">
-          <plugin>mock_components/GenericSystem</plugin>
-          <param name="mock_sensor_commands">${mock_sensor_commands}</param>
-        </xacro:if>
-        <xacro:if value="${sim_gazebo_classic}">
-          <plugin>gazebo_ros2_control/GazeboSystem</plugin>
-        </xacro:if>
-        <xacro:if value="${sim_gazebo}">
-          <plugin>ign_ros2_control/IgnitionSystem</plugin>
-        </xacro:if>
-        <xacro:unless value="${use_mock_hardware or sim_gazebo_classic or sim_gazebo}">
-          <plugin>robot_hardware_inteface/RobotHardwareInteface</plugin>
-        </xacro:unless>
-      </hardware>
-      <joint name="${prefix}rr_wheel">
-        <command_interface name="velocity">
-          <param name="min">-10</param>
-          <param name="max">10</param>
-        </command_interface>
-        <state_interface name="position"/>
-        <state_interface name="velocity"/>
-      </joint>
-      <joint name="${prefix}joint2">
-        <command_interface name="velocity">
-          <param name="min">-10</param>
-          <param name="max">10</param>
-        </command_interface>
-        <state_interface name="position"/>
-        <state_interface name="velocity"/>
-      </joint>
-      <joint name="${prefix}joint3">
-        <command_interface name="velocity">
-          <param name="min">-10</param>
-          <param name="max">10</param>
-        </command_interface>
-        <state_interface name="position"/>
-        <state_interface name="velocity"/>
-      </joint>
-      <joint name="${prefix}joint4">
-        <command_interface name="velocity">
-          <param name="min">-10</param>
-          <param name="max">10</param>
-        </command_interface>
-        <state_interface name="position"/>
-        <state_interface name="velocity"/>
-      </joint>
-    </ros2_control>
-    <xacro:if value="$(arg sim_gazebo_classic)">
-      <!-- Gazebo plugins -->
-      <gazebo reference="world">
-      </gazebo>
-      <gazebo>
-        <plugin filename="libgazebo_ros2_control.so" name="gazebo_ros2_control">
-          <parameters>${simulation_controllers}</parameters>
-        </plugin>
-      </gazebo>
-    </xacro:if>
-    <xacro:if value="$(arg sim_gazebo)">
-      <!-- Gazebo plugins -->
-      <gazebo reference="world">
-      </gazebo>
-      <gazebo>
-        <plugin filename="libign_ros2_control-system.so" name="ign_ros2_control::IgnitionROS2ControlPlugin">
-          <parameters>${simulation_controllers}</parameters>
-          <controller_manager_node_name>${prefix}controller_manager</controller_manager_node_name>
-        </plugin>
-      </gazebo>
-    </xacro:if>
-  </xacro:macro>
+  <ros2_control name="GazeboSystem" type="system">
+    <hardware>
+        <plugin>gazebo_ros2_control/GazeboSystem</plugin>
+    </hardware>
+    <joint name="rf_wheel">
+      <command_interface name="velocity">
+        <param name="min">-10</param>
+        <param name="max">10</param>
+      </command_interface>
+      <state_interface name="position"/>
+      <state_interface name="velocity"/>
+    </joint>
+    <joint name="$fl_wheel">
+      <command_interface name="velocity">
+        <param name="min">-10</param>
+        <param name="max">10</param>
+      </command_interface>
+      <state_interface name="position"/>
+      <state_interface name="velocity"/>
+    </joint>
+    <!-- NOTE the following commented out while implementing front wheels -->
+    <!-- <joint name="${prefix}rr_wheel">
+      <command_interface name="velocity">
+        <param name="min">-10</param>
+        <param name="max">10</param>
+      </command_interface>
+      <state_interface name="position"/>
+      <state_interface name="velocity"/>
+    </joint>
+    <joint name="${prefix}rl_wheel">
+      <command_interface name="velocity">
+        <param name="min">-10</param>
+        <param name="max">10</param>
+      </command_interface>
+      <state_interface name="position"/>
+      <state_interface name="velocity"/>
+    </joint> -->
+  </ros2_control>
+  <gazebo>
+    <plugin filename="libgazebo_ros2_control.so" name="gazebo_ros2_control">
+      <parameters>$(find catbot_description)/config/controllers.yaml</parameters>
+      <parameters>$(find catbot_description)/config/gazebo_ros2_ctl_use_sim.yaml</parameters>
+    </plugin>
+  </gazebo>
 </robot>

Commit message: gazebo_ros2_control launches

File: src/catbot_description/urdf/catbot.urdf.xacro (robot description, xacro)
@@ -13,15 +13,3 @@
     <xacro:include filename="gazebo_control.xacro" />
   </xacro:unless>
-  <!-- Load robot's macro with parameters -->
-  <!-- set prefix if multiple robots are used -->
-  <!-- <xacro:if value="$(arg use_ros2_control)"> -->
-    <!-- <xacro:catbot_ros2_control
-      name="catbot"
-      prefix="$(arg prefix)"
-      use_mock_hardware="$(arg use_mock_hardware)"
-      mock_sensor_commands="$(arg mock_sensor_commands)"
-      sim_gazebo_classic="$(arg sim_gazebo_classic)"
-      sim_gazebo="$(arg sim_gazebo)"
-      simulation_controllers="$(arg simulation_controllers)" /> -->
-  <!-- </xacro:if>  -->
 </robot>

File: src/catbot_description/urdf/catbot/catbot_macro.ros2_control.xacro (robot description, xacro)
@@ -1,42 +1,42 @@
 <?xml version="1.0" encoding="UTF-8"?>
 <robot xmlns:xacro="http://wiki.ros.org/xacro">
-  <ros2_control name="GazeboSystem" type="system">
-    <hardware>
-        <plugin>gazebo_ros2_control/GazeboSystem</plugin>
-    </hardware>
-    <joint name="rf_wheel">
-      <command_interface name="velocity">
-        <param name="min">-10</param>
-        <param name="max">10</param>
-      </command_interface>
-      <state_interface name="position"/>
-      <state_interface name="velocity"/>
-    </joint>
-    <joint name="$fl_wheel">
-      <command_interface name="velocity">
-        <param name="min">-10</param>
-        <param name="max">10</param>
-      </command_interface>
-      <state_interface name="position"/>
-      <state_interface name="velocity"/>
-    </joint>
-    <!-- NOTE the following commented out while implementing front wheels -->
-    <!-- <joint name="${prefix}rr_wheel">
-      <command_interface name="velocity">
-        <param name="min">-10</param>
-        <param name="max">10</param>
-      </command_interface>
-      <state_interface name="position"/>
-      <state_interface name="velocity"/>
-    </joint>
-    <joint name="${prefix}rl_wheel">
-      <command_interface name="velocity">
-        <param name="min">-10</param>
-        <param name="max">10</param>
-      </command_interface>
-      <state_interface name="position"/>
-      <state_interface name="velocity"/>
-    </joint> -->
-  </ros2_control>
+    <ros2_control name="GazeboSystem" type="system">
+        <hardware>
+            <plugin>gazebo_ros2_control/GazeboSystem</plugin>
+        </hardware>
+        <joint name="rf_wheel">
+            <command_interface name="velocity">
+                <param name="min">-10</param>
+                <param name="max">10</param>
+            </command_interface>
+            <state_interface name="position"/>
+            <state_interface name="velocity"/>
+        </joint>
+        <joint name="fl_wheel">
+            <command_interface name="velocity">
+                <param name="min">-10</param>
+                <param name="max">10</param>
+            </command_interface>
+            <state_interface name="position"/>
+            <state_interface name="velocity"/>
+        </joint>
+        <!-- NOTE the following commented out while implementing front wheels -->
+        <!-- <joint name="${prefix}rr_wheel">
+        <command_interface name="velocity">
+            <param name="min">-10</param>
+            <param name="max">10</param>
+        </command_interface>
+        <state_interface name="position"/>
+        <state_interface name="velocity"/>
+        </joint>
+        <joint name="${prefix}rl_wheel">
+        <command_interface name="velocity">
+            <param name="min">-10</param>
+            <param name="max">10</param>
+        </command_interface>
+        <state_interface name="position"/>
+        <state_interface name="velocity"/>
+        </joint> -->
+    </ros2_control>
     <gazebo>
         <plugin name='gazebo_ros2_control' filename='libgazebo_ros2_control.so'>

Commit message: Feature/ros2 control sim (#27)
* Use gazebo_ros2_control

* approximate wheel collision as spheres to fix gazebo bug

* align Gazebo and RViz model

* make sim args work

* rviz camera angle to follow robot

* update README.md with simulation info

* add catbot_simulation to CI linting

File: src/catbot_description/urdf/catbot.urdf.xacro (robot description, xacro)
@@ -3,10 +3,6 @@
   <!-- Use this if parameters are set from the launch file, otherwise delete -->
   <xacro:arg name="prefix" default="" />
-  <xacro:arg name="use_ros2_control" default="false"/>
-  <xacro:arg name="use_mock_hardware" default="false" />
-  <xacro:arg name="mock_sensor_commands" default="false" />
-  <xacro:arg name="sim_gazebo_classic" default="false" />
-  <xacro:arg name="sim_gazebo" default="false" />
-  <xacro:arg name="simulation_controllers" default="" />
+  <xacro:arg name="use_ros2_control" default="true"/>
+  <xacro:arg name="sim_mode" default="false"/>
   <xacro:include filename="$(find catbot_description)/urdf/catbot/catbot_macro.xacro"/>
   <xacro:include filename="gazebo_catbot.xacro" />
@@ -17,15 +13,3 @@
     <xacro:include filename="gazebo_control.xacro" />
   </xacro:unless>
-  <!-- Load robot's macro with parameters -->
-  <!-- set prefix if multiple robots are used -->
-  <xacro:if value="$(arg use_ros2_control)">
-    <xacro:catbot_ros2_control
-      name="catbot"
-      prefix="$(arg prefix)"
-      use_mock_hardware="$(arg use_mock_hardware)"
-      mock_sensor_commands="$(arg mock_sensor_commands)"
-      sim_gazebo_classic="$(arg sim_gazebo_classic)"
-      sim_gazebo="$(arg sim_gazebo)"
-      simulation_controllers="$(arg simulation_controllers)" />
-  </xacro:if>
 </robot>

File: src/catbot_description/urdf/catbot/catbot_macro.ros2_control.xacro (robot description, xacro)
@@ -1,83 +1,49 @@
 <?xml version="1.0" encoding="UTF-8"?>
 <robot xmlns:xacro="http://wiki.ros.org/xacro">
-  <xacro:macro name="catbot_ros2_control" params="
-               name
-               prefix
-               use_mock_hardware:=^|false
-               mock_sensor_commands:=^|false
-               sim_gazebo_classic:=^|false
-               sim_gazebo:=^|false
-               simulation_controllers"
-               >
-    <ros2_control name="${name}" type="system">
-      <hardware>
-        <xacro:if value="${use_mock_hardware}">
-          <plugin>mock_components/GenericSystem</plugin>
-          <param name="mock_sensor_commands">${mock_sensor_commands}</param>
-        </xacro:if>
-        <xacro:if value="${sim_gazebo_classic}">
-          <plugin>gazebo_ros2_control/GazeboSystem</plugin>
-        </xacro:if>
-        <xacro:if value="${sim_gazebo}">
-          <plugin>ign_ros2_control/IgnitionSystem</plugin>
-        </xacro:if>
-        <xacro:unless value="${use_mock_hardware or sim_gazebo_classic or sim_gazebo}">
-          <plugin>robot_hardware_inteface/RobotHardwareInteface</plugin>
-        </xacro:unless>
-      </hardware>
-      <joint name="${prefix}rr_wheel">
+    <ros2_control name="GazeboSystem" type="system">
+        <hardware>
+            <plugin>gazebo_ros2_control/GazeboSystem</plugin>
+        </hardware>
+        <joint name="rf_wheel">
+            <command_interface name="velocity">
+                <param name="min">-10</param>
+                <param name="max">10</param>
+            </command_interface>
+            <state_interface name="position"/>
+            <state_interface name="velocity"/>
+        </joint>
+        <joint name="fl_wheel">
+            <command_interface name="velocity">
+                <param name="min">-10</param>
+                <param name="max">10</param>
+            </command_interface>
+            <state_interface name="position"/>
+            <state_interface name="velocity"/>
+        </joint>
+        <!-- NOTE the following commented out while implementing front wheels -->
+        <!-- <joint name="${prefix}rr_wheel">
         <command_interface name="velocity">
-          <param name="min">-10</param>
-          <param name="max">10</param>
+            <param name="min">-10</param>
+            <param name="max">10</param>
         </command_interface>
         <state_interface name="position"/>
         <state_interface name="velocity"/>
-      </joint>
-      <joint name="${prefix}joint2">
+        </joint>
+        <joint name="${prefix}rl_wheel">
         <command_interface name="velocity">
-          <param name="min">-10</param>
-          <param name="max">10</param>
+            <param name="min">-10</param>
+            <param name="max">10</param>
         </command_interface>
         <state_interface name="position"/>
         <state_interface name="velocity"/>
-      </joint>
-      <joint name="${prefix}joint3">
-        <command_interface name="velocity">
-          <param name="min">-10</param>
-          <param name="max">10</param>
-        </command_interface>
-        <state_interface name="position"/>
-        <state_interface name="velocity"/>
-      </joint>
-      <joint name="${prefix}joint4">
-        <command_interface name="velocity">
-          <param name="min">-10</param>
-          <param name="max">10</param>
-        </command_interface>
-        <state_interface name="position"/>
-        <state_interface name="velocity"/>
-      </joint>
+        </joint> -->
     </ros2_control>
-    <xacro:if value="$(arg sim_gazebo_classic)">
-      <!-- Gazebo plugins -->
-      <gazebo reference="world">
-      </gazebo>
-      <gazebo>
-        <plugin filename="libgazebo_ros2_control.so" name="gazebo_ros2_control">
-          <parameters>${simulation_controllers}</parameters>
+    <gazebo>
+        <plugin name='gazebo_ros2_control' filename='libgazebo_ros2_control.so'>
+            <robot_param>robot_description</robot_param>
+            <robot_param_node>robot_state_publisher</robot_param_node>
+            <parameters>$(find catbot_description)/config/controllers.yaml</parameters>
+            <!-- <parameters>$(find catbot_description)/config/gazebo_ros2_ctl_use_sim.yaml</parameters> -->
         </plugin>
-      </gazebo>
-    </xacro:if>
-    <xacro:if value="$(arg sim_gazebo)">
-      <!-- Gazebo plugins -->
-      <gazebo reference="world">
-      </gazebo>
-      <gazebo>
-        <plugin filename="libign_ros2_control-system.so" name="ign_ros2_control::IgnitionROS2ControlPlugin">
-          <parameters>${simulation_controllers}</parameters>
-          <controller_manager_node_name>${prefix}controller_manager</controller_manager_node_name>
-        </plugin>
-      </gazebo>
-    </xacro:if>
-  </xacro:macro>
+    </gazebo>
 </robot>

File: src/catbot_description/urdf/catbot/catbot_macro.xacro (robot description, xacro)
@@ -2,9 +2,11 @@
 <robot xmlns:xacro="http://wiki.ros.org/xacro">
   <xacro:include filename="inertial_macros.xacro"/>
+  <xacro:property name="sphere_wheel_offset" value="0.006"/>
   <link name="base_link"></link>
   <joint name="chassis_joint" type="fixed">
     <parent link="base_link" />
     <child link="still_chassis_assm" />
-    <origin rpy="0.0 0 0" xyz="0 0 0" />
+    <!-- rotate 90deg to orient correctly -->
+    <origin rpy="0.0 0 1.5708" xyz="0 0 0" />
   </joint>
   <link name="still_chassis_assm">
@@ -47,7 +49,8 @@
     </visual>
     <collision>
-      <origin xyz="0 0 0" rpy="0 -0 0" />
+      <origin xyz="0 0 -${sphere_wheel_offset}" rpy="0 -0 0" />
       <geometry>
-        <mesh filename="package://catbot_description/meshes/collision/wheel_assm_collision.stl" />
+        <!-- <mesh filename="package://catbot_description/meshes/collision/wheel_assm_collision.stl" /> -->
+        <sphere radius="${wheel_radius}"/>
       </geometry>
     </collision>
@@ -84,7 +87,8 @@
     </visual>
     <collision>
-      <origin xyz="0 0 0" rpy="0 -0 0" />
+      <origin xyz="0 0 -${sphere_wheel_offset}" rpy="0 -0 0" />
       <geometry>
-        <mesh filename="package://catbot_description/meshes/collision/wheel_assm_2_collision.stl" />
+        <!-- <mesh filename="package://catbot_description/meshes/collision/wheel_assm_2_collision.stl" /> -->
+        <sphere radius="${wheel_radius}"/>
       </geometry>
     </collision>
@@ -121,7 +125,8 @@
     </visual>
     <collision>
-      <origin xyz="0 0 0" rpy="0 -0 0" />
+      <origin xyz="0 0 -${sphere_wheel_offset}" rpy="0 -0 0" />
       <geometry>
-        <mesh filename="package://catbot_description/meshes/collision/wheel_assm_3_collision.stl" />
+        <!-- <mesh filename="package://catbot_description/meshes/collision/wheel_assm_3_collision.stl" /> -->
+        <sphere radius="${wheel_radius}"/>
       </geometry>
     </collision>
@@ -149,5 +154,5 @@
   <link name="wheel_assm_4">
     <visual>
-      <origin xyz="0 0 0" rpy="0 -0 0" />
+      <origin xyz="0 0 ${sphere_wheel_offset}" rpy="0 -0 0" />
       <geometry>
         <mesh filename="package://catbot_description/meshes/visual/wheel_assm_4_visual.stl" />
@@ -160,5 +165,6 @@
       <origin xyz="0 0 0" rpy="0 -0 0" />
       <geometry>
-        <mesh filename="package://catbot_description/meshes/collision/wheel_assm_4_collision.stl" />
+        <!-- <mesh filename="package://catbot_description/meshes/collision/wheel_assm_4_collision.stl" /> -->
+        <sphere radius="${wheel_radius}"/>
       </geometry>
     </collision>

Commit message: scheme similar to linorobot2

File: src/catbot_description/urdf/catbot.urdf.xacro (robot description, xacro)
@@ -3,13 +3,18 @@
   <!-- Use this if parameters are set from the launch file, otherwise delete -->
   <xacro:arg name="prefix" default="" />
-  <xacro:arg name="use_ros2_control" default="true"/>
-  <xacro:arg name="sim_mode" default="false"/>
+  <!-- <xacro:arg name="use_ros2_control" default="true"/>
+  <xacro:arg name="sim_mode" default="false"/> -->
   <xacro:include filename="$(find catbot_description)/urdf/catbot/catbot_macro.xacro"/>
   <xacro:include filename="gazebo_catbot.xacro" />
-  <xacro:if value="$(arg use_ros2_control)">
+  <xacro:include filename="4wd_control.xacro"/>
+  <!-- <xacro:if value="$(arg use_ros2_control)">
     <xacro:include filename="$(find catbot_description)/urdf/catbot/catbot_macro.ros2_control.xacro"/>
   </xacro:if>
   <xacro:unless value="$(arg use_ros2_control)">
     <xacro:include filename="gazebo_control.xacro" />
-  </xacro:unless>
+  </xacro:unless> -->
+  <xacro:diff_drive_controller
+    wheel_separation="${0.156}"
+    wheel_diameter="${0.066}"
+  />
 </robot>

File: src/catbot_description/urdf/catbot/catbot_macro.xacro (robot description, xacro)
@@ -67,5 +67,5 @@
       </inertial>
   </link>
-  <joint name="rr_wheel" type="fixed">
+  <joint name="rr_wheel" type="continuous">
     <origin xyz="-0.077614131532514007983 0.080478921592024327269 -0.030500000000000013212"
     rpy="-1.570796326794896558 0.67540343776289657463 -1.5707963267948956698" />
@@ -73,6 +73,4 @@
     <child link="wheel_assm" />
     <axis xyz="0 0 1" />
-    <!-- <limit effort="1" velocity="20" />
-    <joint_properties friction="0.0" /> -->
   </joint>
   <link name="wheel_assm_2">
@@ -111,6 +109,4 @@
     <child link="wheel_assm_2" />
     <axis xyz="0 0 1" />
-    <limit effort="1" velocity="20" />
-    <joint_properties friction="0.0" />
   </joint>
   <link name="wheel_assm_3">
@@ -143,5 +139,5 @@
     </inertial>
   </link>
-  <joint name="rl_wheel" type="fixed">
+  <joint name="rl_wheel" type="continuous">
     <origin xyz="0.078385868467483257871 0.080478921592024507681 -0.030500000000000044437"
     rpy="-1.570796326794896558 -5.0445758681405660746e-15 1.5707963267948970021" />
@@ -149,6 +145,4 @@
     <child link="wheel_assm_3" />
     <axis xyz="0 0 1" />
-    <!-- <limit effort="1" velocity="20" />
-    <joint_properties friction="0.0" /> -->
   </joint>
   <link name="wheel_assm_4">
@@ -187,6 +181,4 @@
     <child link="wheel_assm_4" />
     <axis xyz="0 0 -1" />
-    <limit effort="1" velocity="20" />
-    <joint_properties friction="0.0" />
   </joint>
 </robot>
