Commit message: bastardized linorobot2

File: src/catbot_description/urdf/catbot.urdf.xacro (robot description, xacro)
@@ -1,20 +1,66 @@
-<?xml version="1.0" encoding="UTF-8"?>
-<robot xmlns:xacro="http://wiki.ros.org/xacro" name="catbot">
-  <!-- Use this if parameters are set from the launch file, otherwise delete -->
-  <xacro:arg name="prefix" default="" />
-  <!-- <xacro:arg name="use_ros2_control" default="true"/>
-  <xacro:arg name="sim_mode" default="false"/> -->
-  <xacro:include filename="$(find catbot_description)/urdf/catbot/catbot_macro.xacro"/>
-  <xacro:include filename="gazebo_catbot.xacro" />
-  <xacro:include filename="4wd_control.xacro"/>
-  <!-- <xacro:if value="$(arg use_ros2_control)">
-    <xacro:include filename="$(find catbot_description)/urdf/catbot/catbot_macro.ros2_control.xacro"/>
-  </xacro:if>
-  <xacro:unless value="$(arg use_ros2_control)">
-    <xacro:include filename="gazebo_control.xacro" />
-  </xacro:unless> -->
+<?xml version="1.0"?>
+<robot name="catbot_4wd" xmlns:xacro="http://ros.org/wiki/xacro">
+  <xacro:include filename="$(find catbot_description)/urdf/4wd_properties.urdf.xacro" />
+  <xacro:include filename="$(find catbot_description)/urdf/mech/base.urdf.xacro" />
+  <xacro:include filename="$(find catbot_description)/urdf/mech/wheel.urdf.xacro" />
+  <!-- <xacro:include filename="$(find catbot_description)/urdf/sensors/imu.urdf.xacro" />
+  <xacro:include filename="$(find catbot_description)/urdf/sensors/generic_laser.urdf.xacro" />
+  <xacro:include filename="$(find catbot_description)/urdf/sensors/depth_sensor.urdf.xacro" /> -->
+  <xacro:include filename="$(find catbot_description)/urdf/controllers/skid_steer.urdf.xacro" />
+  <xacro:base
+    length="${base_length}"
+    width="${base_width}"
+    height="${base_height}"
+    mass="${base_mass}"
+    wheel_radius="${wheel_radius}"
+    wheel_pos_z="${wheel_pos_z}"
+/>
+  <xacro:wheel
+    side="front_left"
+    radius="${wheel_radius}"
+    width="${wheel_width}"
+    pos_x="${wheel_pos_x}"
+    pos_y="${wheel_pos_y}"
+    pos_z="${wheel_pos_z}"
+    mass="${wheel_mass}"
+  />
+  <xacro:wheel
+    side="front_right"
+    radius="${wheel_radius}"
+    width="${wheel_width}"
+    pos_x="${wheel_pos_x}"
+    pos_y="${-wheel_pos_y}"
+    pos_z="${wheel_pos_z}"
+    mass="${wheel_mass}"
+  />
+  <xacro:wheel
+    side="rear_left"
+    radius="${wheel_radius}"
+    width="${wheel_width}"
+    pos_x="${-wheel_pos_x}"
+    pos_y="${wheel_pos_y}"
+    pos_z="${wheel_pos_z}"
+    mass="${wheel_mass}"
+  />
+  <xacro:wheel
+    side="rear_right"
+    radius="${wheel_radius}"
+    width="${wheel_width}"
+    pos_x="${-wheel_pos_x}"
+    pos_y="${-wheel_pos_y}"
+    pos_z="${wheel_pos_z}"
+    mass="${wheel_mass}"
+  />
+  <!-- <xacro:imu/>
+  <xacro:generic_laser>
+    <xacro:insert_block name="laser_pose" />
+  </xacro:generic_laser>
+  <xacro:depth_sensor>
+    <xacro:insert_block name="depth_sensor_pose" />
+  </xacro:depth_sensor> -->
   <xacro:diff_drive_controller
-    wheel_separation="${0.156}"
-    wheel_diameter="${0.066}"
+    wheel_separation="${wheel_pos_y * 2}"
+    wheel_radius="${wheel_radius}"
+    wheel_torque="${wheel_torque}"
   />
 </robot>

File: src/catbot_description/urdf/catbot/catbot_macro.xacro (robot description, xacro)
@@ -87,5 +87,5 @@
     <child link="wheel_assm" />
     <axis xyz="0 0 1" />
-    <limit effort="1" velocity="20" />
+    <!-- <limit effort="1" velocity="20" /> -->
   </joint>
   <link name="wheel_assm_2">
@@ -134,5 +134,5 @@
     <child link="wheel_assm_2" />
     <axis xyz="0 0 1" />
-    <limit effort="1" velocity="20" />
+    <!-- <limit effort="1" velocity="20" /> -->
   </joint>
   <link name="wheel_assm_3">
@@ -181,5 +181,5 @@
     <child link="wheel_assm_3" />
     <axis xyz="0 0 1" />
-    <limit effort="1" velocity="20" />
+    <!-- <limit effort="1" velocity="20" /> -->
   </joint>
   <link name="wheel_assm_4">
@@ -228,5 +228,5 @@
     <child link="wheel_assm_4" />
     <axis xyz="0 0 -1" />
-    <limit effort="1" velocity="20" />
+    <!-- <limit effort="1" velocity="20" /> -->
   </joint>
 </robot>

File: src/catbot_description/urdf/catbot/inertial_macros.xacro (robot description, xacro)
@@ -25,7 +25,7 @@
             <xacro:insert_block name="origin"/>
             <mass value="${mass}" />
-            <inertia ixx="${(1/12) * mass * (3*radius*radius + length*length)}" ixy="0.0" ixz="0.0"
-                    iyy="${(1/12) * mass * (3*radius*radius + length*length)}" iyz="0.0"
-                    izz="${(1/2) * mass * (radius*radius)}" />
+            <inertia ixx="${(2/5) * mass * (radius * radius)}" ixy="0" ixz="0"
+                 iyy="${(2/5) * mass * (radius * radius)}" iyz="0"
+                 izz="${(2/5) * mass * (radius * radius)}" />
         </inertial>
     </xacro:macro>

File: src/catbot_description/urdf/controllers/skid_steer.urdf.xacro (robot description, xacro)
@@ -1,4 +1,4 @@
-<robot xmlns:xacro="http://www.ros.org/wiki/xacro">
-  <xacro:macro name="diff_drive_controller" params="wheel_separation wheel_diameter">
+<robot xmlns:xacro="http://ros.org/wiki/xacro">
+  <xacro:macro name="diff_drive_controller" params="wheel_separation wheel_radius wheel_torque">
     <gazebo>
       <plugin name="differential_drive_controller" filename="libgazebo_ros_diff_drive.so">
@@ -7,5 +7,4 @@
         </ros>
         <num_wheel_pairs>2</num_wheel_pairs>
-        <!-- Wheel Information -->
         <left_joint>front_left_wheel_joint</left_joint>
         <right_joint>front_right_wheel_joint</right_joint>
@@ -14,15 +13,13 @@
         <wheel_separation>${wheel_separation}</wheel_separation>
         <wheel_separation>${wheel_separation}</wheel_separation>
-        <wheel_diameter>${wheel_diameter}</wheel_diameter>
-        <wheel_diameter>${wheel_diameter}</wheel_diameter>
-        <!-- Limits -->
+        <wheel_diameter>${wheel_radius * 2}</wheel_diameter>
+        <wheel_diameter>${wheel_radius * 2}</wheel_diameter>
         <updateRate>100</updateRate>
         <max_wheel_acceleration>1.0</max_wheel_acceleration>
-        <!-- Output -->
-        <odometry_frame>odom</odometry_frame>
-        <robot_base_frame>base_link</robot_base_frame>
-        <publish_odom>false</publish_odom>
+        <robot_base_frame>base_footprint</robot_base_frame>
+        <publish_odom>true</publish_odom>
         <publish_odom_tf>false</publish_odom_tf>
         <publish_wheel_tf>true</publish_wheel_tf>
+        <odometry_frame>odom</odometry_frame>
       </plugin>
     </gazebo>

File: src/catbot_description/urdf/gazebo_catbot.xacro (robot description, xacro)
@@ -2,8 +2,8 @@
 <robot xmlns:xacro="http://ros.org/wiki/xacro">
     <xacro:macro name="gz_wheel_physics">
-        <!-- <mu1 value="1.0"/>
-        <mu2 value="0.5"/>
-        <kp value="10000000.0"/>
-        <kd value="1.0"/> -->
+        <!-- <mu1 value="1.0"/> -->
+        <!-- <mu2 value="0.5"/> -->
+        <!-- <kp value="10000000.0"/> -->
+        <!-- <kd value="1.0"/> -->
         <!-- <fdir1 value="1 0 0"/> -->
     </xacro:macro>
