Commit message: broken verison of mesh support

File: src/catbot_description/urdf/4wd_properties.urdf.xacro (robot description, xacro)
@@ -3,6 +3,6 @@
   <xacro:property name="base_length" value="0.242" />
   <xacro:property name="base_width" value="0.126" />
-  <xacro:property name="base_height" value="0.064" />
-  <xacro:property name="base_mass" value="1.015" />
+  <xacro:property name="base_height" value="0.09368130" />
+  <xacro:property name="base_mass" value="1.016" />
   <xacro:property name="wheel_radius" value="0.033" />
   <xacro:property name="wheel_width" value="0.0265" />

File: src/catbot_description/urdf/catbot.urdf.xacro (robot description, xacro)
@@ -24,4 +24,5 @@
     pos_z="${wheel_pos_z}"
     mass="${wheel_mass}"
+    visual_yaw="0"
   />
   <xacro:wheel
@@ -33,4 +34,5 @@
     pos_z="${wheel_pos_z}"
     mass="${wheel_mass}"
+    visual_yaw="${pi}"
   />
   <xacro:wheel
@@ -42,4 +44,5 @@
     pos_z="${wheel_pos_z}"
     mass="${wheel_mass}"
+    visual_yaw="0"
   />
   <xacro:wheel
@@ -51,4 +54,5 @@
     pos_z="${wheel_pos_z}"
     mass="${wheel_mass}"
+    visual_yaw="${pi}"
   />
   <!-- <xacro:imu/>

File: src/catbot_description/urdf/mech/base.urdf.xacro (robot description, xacro)
@@ -5,12 +5,12 @@
     <link name="base_link">
       <visual>
-        <origin xyz="0 0 0" rpy="0 0 0"/>
+        <origin xyz="0 0 0" rpy="0 0 1.57"/>
         <geometry>
-          <box size="${length} ${width} ${height}"/>
-          <!-- <mesh filename="" scale="0.001 0.001 0.001"/> -->
+          <!-- <box size="${length} ${width} ${height}"/> -->
+          <mesh filename="file://$(find catbot_description)/meshes/visual/still_chassis_assm_visual.stl"/>
         </geometry>
-        <material name="yellow">
-          <color rgba="0.8784 0.6627 0.6627 1.0"/>
-        </material>
+        <material name="still_chassis_assm_material">
+        <color rgba="0.66987717125153911635 0.81712318213796708566 0.66602980483018847657 1.0" />
+      </material>
       </visual>
       <collision>
@@ -29,12 +29,5 @@
     </link>
     <gazebo reference="base_link">
-      <visual>
-        <material>
-          <ambient>0.8392 0.6314 0.0 1.0</ambient>
-          <diffuse>0.8392 0.6314 0.0 1.0</diffuse>
-          <specular>0.99 0.99 0.99 1.0</specular>
-          <emissive>0.0 0.0 0.0 0.0</emissive>
-        </material>
-      </visual>
+      <material>Gazebo/Green</material>
     </gazebo>
     <joint name="base_to_footprint" type="fixed">

File: src/catbot_description/urdf/mech/wheel.urdf.xacro (robot description, xacro)
@@ -1,14 +1,18 @@
 <?xml version="1.0"?>
 <robot xmlns:xacro="http://ros.org/wiki/xacro">
-  <xacro:macro name="wheel" params="side radius width pos_x pos_y pos_z mass">
+  <xacro:macro name="wheel" params="side radius width pos_x pos_y pos_z mass visual_yaw">
     <link name="${side}_wheel_link">
       <visual>
-        <origin xyz="0 0 0" rpy="${pi/2} 0 0"/>
+        <origin xyz="0 0 0" rpy="${pi/2} 0 ${visual_yaw}"/>
+        <geometry>
+          <mesh filename="file://$(find catbot_description)/meshes/visual/wheel_assm_visual.stl"/>
+        </geometry>
+        <!-- <origin xyz="0 0 0" rpy="${pi/2} 0 0"/>
         <geometry>
           <cylinder radius="${radius}" length="${width}"/>
-        </geometry>
-        <material name="blue">
-            <color rgba="0.1764 0.4588 0.8509 1.0"/>
-        </material>
+        </geometry> -->
+        <material name="wheel_assm_material">
+        <color rgba="0.34876043041436377568 0.28454440741211711741 0.12249285133838178075 1.0" />
+      </material>
       </visual>
       <collision>
@@ -27,12 +31,5 @@
     </link>
     <gazebo reference="${side}_wheel_link">
-      <visual>
-        <material>
-          <ambient>0.1764 0.4588 0.8509 1.0</ambient>
-          <diffuse>0.1764 0.4588 0.8509 1.0</diffuse>
-          <specular>0.1764 0.4588 0.8509 1.0</specular>
-          <emissive>0.0 0.0 0.0 0.0</emissive>
-        </material>
-      </visual>
+      <material>Gazebo/Black</material>
     </gazebo>
     <joint name="${side}_wheel_joint" type="continuous">

Commit message: fixed wheel positions in space

File: src/catbot_description/urdf/4wd_properties.urdf.xacro (robot description, xacro)
@@ -8,8 +8,10 @@
   <xacro:property name="wheel_width" value="0.0265" />
   <xacro:property name="wheel_pos_x" value="0.087" />
-  <xacro:property name="wheel_pos_y" value="0.08" />
-  <xacro:property name="wheel_pos_z" value="-0.06" />
+  <xacro:property name="wheel_pos_y" value="0.07838587" />
+  <xacro:property name="wheel_pos_z" value="-0.0304" />
   <xacro:property name="wheel_mass" value=".054378" />
   <xacro:property name="wheel_torque" value="20" />
+  <xacro:property name="origin_to_front_wheels_x" value="0.06802108" />
+  <xacro:property name="origin_to_rear_wheels_x" value="0.08047892" />
   <xacro:property name="laser_pose">
     <origin xyz="0.0475 0 0.082" rpy="0 0 0"/>

File: src/catbot_description/urdf/catbot.urdf.xacro (robot description, xacro)
@@ -20,5 +20,5 @@
     radius="${wheel_radius}"
     width="${wheel_width}"
-    pos_x="${wheel_pos_x}"
+    pos_x="${origin_to_front_wheels_x}"
     pos_y="${wheel_pos_y}"
     pos_z="${wheel_pos_z}"
@@ -30,5 +30,5 @@
     radius="${wheel_radius}"
     width="${wheel_width}"
-    pos_x="${wheel_pos_x}"
+    pos_x="${origin_to_front_wheels_x}"
     pos_y="${-wheel_pos_y}"
     pos_z="${wheel_pos_z}"
@@ -40,5 +40,5 @@
     radius="${wheel_radius}"
     width="${wheel_width}"
-    pos_x="${-wheel_pos_x}"
+    pos_x="${-origin_to_rear_wheels_x}"
     pos_y="${wheel_pos_y}"
     pos_z="${wheel_pos_z}"
@@ -50,5 +50,5 @@
     radius="${wheel_radius}"
     width="${wheel_width}"
-    pos_x="${-wheel_pos_x}"
+    pos_x="${-origin_to_rear_wheels_x}"
     pos_y="${-wheel_pos_y}"
     pos_z="${wheel_pos_z}"

Commit message: fixed y-axis alignment of wheel collision

File: src/catbot_description/urdf/4wd_properties.urdf.xacro (robot description, xacro)
@@ -5,6 +5,10 @@
   <xacro:property name="base_height" value="0.09368130" />
   <xacro:property name="base_mass" value="1.016" />
-  <xacro:property name="wheel_radius" value="0.033" />
+  <xacro:property name="wheel_radius" value="${0.00240839 + 0.03150000}" />
   <xacro:property name="wheel_width" value="0.0265" />
+  <xacro:property name="wheel_assembly_width" value="0.03140000"/>
+  <!-- not sure why this is needed, but makes collision line up with vidual -->
+  <xacro:property name="wheel_collision_offset_correction" value="0.002"/>
+  <xacro:property name="wheel_collision_offset" value="${wheel_collision_offset_correction + wheel_assembly_width - wheel_width}"/>
   <xacro:property name="wheel_pos_x" value="0.087" />
   <xacro:property name="wheel_pos_y" value="0.07838587" />

File: src/catbot_description/urdf/catbot.urdf.xacro (robot description, xacro)
@@ -20,4 +20,5 @@
     radius="${wheel_radius}"
     width="${wheel_width}"
+    collision_offset="${wheel_collision_offset}"
     pos_x="${origin_to_front_wheels_x}"
     pos_y="${wheel_pos_y}"
@@ -30,4 +31,5 @@
     radius="${wheel_radius}"
     width="${wheel_width}"
+    collision_offset="${-wheel_collision_offset}"
     pos_x="${origin_to_front_wheels_x}"
     pos_y="${-wheel_pos_y}"
@@ -40,4 +42,5 @@
     radius="${wheel_radius}"
     width="${wheel_width}"
+    collision_offset="${wheel_collision_offset}"
     pos_x="${-origin_to_rear_wheels_x}"
     pos_y="${wheel_pos_y}"
@@ -50,4 +53,5 @@
     radius="${wheel_radius}"
     width="${wheel_width}"
+    collision_offset="${-wheel_collision_offset}"
     pos_x="${-origin_to_rear_wheels_x}"
     pos_y="${-wheel_pos_y}"

File: src/catbot_description/urdf/mech/wheel.urdf.xacro (robot description, xacro)
@@ -1,5 +1,5 @@
 <?xml version="1.0"?>
 <robot xmlns:xacro="http://ros.org/wiki/xacro">
-  <xacro:macro name="wheel" params="side radius width pos_x pos_y pos_z mass visual_yaw">
+  <xacro:macro name="wheel" params="side radius width collision_offset pos_x pos_y pos_z mass visual_yaw">
     <link name="${side}_wheel_link">
       <visual>
@@ -17,5 +17,5 @@
       </visual>
       <collision>
-        <origin xyz="0 0 0" rpy="${pi/2} 0 0"/>
+        <origin xyz="0 ${collision_offset} 0" rpy="${pi/2} 0 0"/>
         <geometry>
           <cylinder radius="${radius}" length="${width}"/>
