Commit message: update from onshape again

File: src/catbot_description/onshape/catbot/robot.urdf (robot description, URDF)
Before this commit: robot catbot, 6 links, 5 joints
Links:
- link still_chassis_assm: mass 1.0156681416365394011 -> 1.015668141636539179

File: src/catbot_description/urdf/catbot.urdf.xacro (robot description, xacro)
@@ -3,4 +3,5 @@
   <!-- Use this if parameters are set from the launch file, otherwise delete -->
   <xacro:arg name="prefix" default="" />
+  <xacro:arg name="use_ros2_control" default="false"/>
   <xacro:arg name="use_mock_hardware" default="false" />
   <xacro:arg name="mock_sensor_commands" default="false" />
@@ -9,6 +10,11 @@
   <xacro:arg name="simulation_controllers" default="" />
   <xacro:include filename="$(find catbot_description)/urdf/catbot/catbot_macro.xacro"/>
-  <xacro:include filename="$(find catbot_description)/urdf/catbot/catbot_macro.ros2_control.xacro"/>
-  <xacro:include filename="gazebo_catbot.xacro"/>
+  <xacro:include filename="gazebo_catbot.xacro" />
+  <xacro:if value="$(arg use_ros2_control)">
+    <xacro:include filename="$(find catbot_description)/urdf/catbot/catbot_macro.ros2_control.xacro"/>
+  </xacro:if>
+  <xacro:unless value="$(arg use_ros2_control)">
+    <xacro:include filename="gazebo_control.xacro" />
+  </xacro:unless>
   <!-- create link fixed to the "world" -->
   <link name="world" />
@@ -18,11 +24,13 @@
     <origin xyz="0 0 0.0635" rpy="0 0 0" />          <!-- position robot in the world -->
   </xacro:catbot>
-  <xacro:catbot_ros2_control
-    name="catbot"
-    prefix="$(arg prefix)"
-    use_mock_hardware="$(arg use_mock_hardware)"
-    mock_sensor_commands="$(arg mock_sensor_commands)"
-    sim_gazebo_classic="$(arg sim_gazebo_classic)"
-    sim_gazebo="$(arg sim_gazebo)"
-    simulation_controllers="$(arg simulation_controllers)" />
+  <xacro:if value="$(arg use_ros2_control)">
+    <xacro:catbot_ros2_control
+      name="catbot"
+      prefix="$(arg prefix)"
+      use_mock_hardware="$(arg use_mock_hardware)"
+      mock_sensor_commands="$(arg mock_sensor_commands)"
+      sim_gazebo_classic="$(arg sim_gazebo_classic)"
+      sim_gazebo="$(arg sim_gazebo)"
+      simulation_controllers="$(arg simulation_controllers)" />
+  </xacro:if>
 </robot>

File: src/catbot_description/urdf/catbot/catbot_macro.xacro (robot description, xacro)
@@ -21,5 +21,5 @@
         </geometry>
         <material name="still_chassis_assm_material">
-          <color rgba="0.66987717125153900533 0.81712318213796708566 0.66602980483018836555 1.0" />
+          <color rgba="0.66987717125153911635 0.81712318213796708566 0.66602980483018847657 1.0" />
         </material>
       </visual>
@@ -31,12 +31,12 @@
       </collision>
       <inertial>
-        <origin xyz="0.00027961412402240977014 0.0046876789374875839009 -0.0054409557585405705568"
+        <origin xyz="0.00027961412402240787278 0.0046876789374875821662 -0.0054409557585405705568"
         rpy="0 0 0" />
-        <mass value="1.0156681416365394011" />
+        <mass value="1.015668141636539179" />
         <inertia ixx="0.0065127126032337098738"
-        ixy="1.5566438777542365468e-07"
-        ixz="3.6708728527239328719e-06"
+        ixy="1.5566438777546685336e-07"
+        ixz="3.6708728527239311778e-06"
         iyy="0.0025991819436423468752"
-        iyz="6.1954470337197489749e-05"
+        iyz="6.1954470337197611722e-05"
         izz="0.0071648278899316356766" />
       </inertial>
@@ -59,12 +59,12 @@
       </collision>
       <inertial>
-        <origin xyz="2.5876683231912983522e-09 -2.5321947387836322962e-09 -0.0043217676979120578026"
+        <origin xyz="2.5876683183573441879e-09 -2.5321947361304500679e-09 -0.0043217676979120569353"
         rpy="0 0 0" />
         <mass value="0.054377782220193432439" />
-        <inertia ixx="1.7947780629583350172e-05"
-        ixy="-3.8234084814183779999e-12"
-        ixz="-1.6934852918263056535e-12"
-        iyy="1.7621269066491265109e-05"
-        iyz="-2.0136050751311128972e-12"
+        <inertia ixx="1.7947780629583346784e-05"
+        ixy="-3.8234084819748992999e-12"
+        ixz="-1.6934852924892931359e-12"
+        iyy="1.7621269066491268497e-05"
+        iyz="-2.0136050748759971485e-12"
         izz="2.8213568549230894094e-05" />
       </inertial>
@@ -96,12 +96,12 @@
       </collision>
       <inertial>
-        <origin xyz="2.5876683436570912888e-09 -2.5321947882875150234e-09 -0.0043217676979120907624"
+        <origin xyz="2.5876683388231371246e-09 -2.5321947856343332086e-09 -0.004321767697912089895"
         rpy="0 0 0" />
         <mass value="0.054377782220193432439" />
-        <inertia ixx="1.7947780629583373889e-05"
-        ixy="-3.8234084806256659389e-12"
-        ixz="-1.6934852952780513878e-12"
-        iyy="1.7621269066491271885e-05"
-        iyz="-2.0136050702142612672e-12"
+        <inertia ixx="1.7947780629583370501e-05"
+        ixy="-3.8234084811821872389e-12"
+        ixz="-1.6934852959410392741e-12"
+        iyy="1.7621269066491275274e-05"
+        iyz="-2.013605069932675335e-12"
         izz="2.8213568549230904259e-05" />
       </inertial>
@@ -133,12 +133,12 @@
       </collision>
       <inertial>
-        <origin xyz="2.5876683542375088732e-09 -2.5321947930490429075e-09 -0.0043217676979121003034"
+        <origin xyz="2.5876683494035538817e-09 -2.5321947903698363363e-09 -0.0043217676979121003034"
         rpy="0 0 0" />
         <mass value="0.054377782220193432439" />
-        <inertia ixx="1.7947780629583373889e-05"
-        ixy="-3.8234084806256627077e-12"
-        ixz="-1.6934852942781941971e-12"
-        iyy="1.7621269066491275274e-05"
-        iyz="-2.01360506846477306e-12"
+        <inertia ixx="1.7947780629583370501e-05"
+        ixy="-3.8234084811821831999e-12"
+        ixz="-1.6934852949411820834e-12"
+        iyy="1.7621269066491278662e-05"
+        iyz="-2.0136050682372531551e-12"
         izz="2.8213568549230904259e-05" />
       </inertial>
@@ -170,12 +170,12 @@
       </collision>
       <inertial>
-        <origin xyz="2.5876682744584021363e-09 -2.5321945349340081079e-09 -0.0043217676979121323957"
+        <origin xyz="2.587668269624447972e-09 -2.5321945322547953329e-09 -0.0043217676979121323957"
         rpy="0 0 0" />
         <mass value="0.054377782220193432439" />
-        <inertia ixx="1.7947780629583377277e-05"
-        ixy="-3.8234084820191074185e-12"
-        ixz="-1.6934852985237760372e-12"
-        iyy="1.7621269066491275274e-05"
-        iyz="-2.0136050684267663727e-12"
+        <inertia ixx="1.7947780629583373889e-05"
+        ixy="-3.8234084825756295263e-12"
+        ixz="-1.6934852991867637216e-12"
+        iyy="1.7621269066491278662e-05"
+        iyz="-2.0136050681091290175e-12"
         izz="2.8213568549230907647e-05" />
       </inertial>

File: src/catbot_description/urdf/gazebo_catbot.xacro (robot description, xacro)
@@ -6,4 +6,6 @@
     <gazebo reference="wheel_assm">
         <material>Gazebo/Black</material>
+        <mu1 value="0.001"/>
+        <mu2 value="0.001"/>
     </gazebo>
     <gazebo reference="wheel_assm_2">
@@ -12,4 +14,6 @@
     <gazebo reference="wheel_assm_3">
         <material>Gazebo/Black</material>
+        <mu1 value="0.001"/>
+        <mu2 value="0.001"/>
     </gazebo>
     <gazebo reference="wheel_assm_4">

Commit message: update onshape to robot

File: src/catbot_description/onshape/catbot/robot.urdf (robot description, URDF)
Before this commit: robot catbot, 6 links, 5 joints
Links:
- removed link base_link
- removed link still_chassis_assm
- removed link wheel_assm
- removed link wheel_assm_2
- removed link wheel_assm_3
- removed link wheel_assm_4
- added link still_chassis_assm__list_nl250j021y5bmp_screwless, mass 1.0300000000000000266; collision box size=0.0060000000000000001249 0.014000000000000000291 0.00500000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; collision box size=0.0060000000000000001249 0.014000000000000000291 0.00500000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
- added link wheel_assm__list_7stftxbui3bodm_screwless, mass 0.04950000000000000927; collision cylinder length=0.0060000000000000001249 radius=0.0069282000000000006773; collision cylinder length=0.0060000000000000001249 radius=0.0069282000000000006773
- added link wheel_assm__list_7stftxbui3bodm_screwless_2, mass 0.04950000000000000927; collision cylinder length=0.0060000000000000001249 radius=0.0069282000000000006773; collision cylinder length=0.0060000000000000001249 radius=0.0069282000000000006773
- added link wheel_assm__list_7stftxbui3bodm_screwless_3, mass 0.04950000000000000927; collision cylinder length=0.0060000000000000001249 radius=0.0069282000000000006773; collision cylinder length=0.0060000000000000001249 radius=0.0069282000000000006773
- added link wheel_assm__list_7stftxbui3bodm_screwless_4, mass 0.04950000000000000927; collision cylinder length=0.0060000000000000001249 radius=0.0069282000000000006773; collision cylinder length=0.0060000000000000001249 radius=0.0069282000000000006773
Joints:
- removed joint base_link_to_base
- removed joint fl_wheel
- removed joint rf_wheel
- removed joint rl_wheel
- removed joint rr_wheel
- added joint front_left_wheel_speed: type revolute, parent wheel_assm__list_7stftxbui3bodm_screwless, child still_chassis_assm__list_nl250j021y5bmp_screwless, origin xyz=0.068021078407975790747 0.078385868467486227718 -0.030499999999999919537 rpy=1.570796326794896558 -1.4446015326859761871e-29 9.7144514656760185879e-17, axis 0 0 1, limit effort=1 velocity=20
- added joint front_right_wheel_speed: type revolute, parent still_chassis_assm__list_nl250j021y5bmp_screwless, child wheel_assm__list_7stftxbui3bodm_screwless_2, origin xyz=8.6042284408449631883e-16 -4.0592529337857286009e-16 0.15599999999999991651 rpy=-3.141592653589778017 1.5256589149154761406e-16 1.5377205745436968165, axis 0 0 1, limit effort=1 velocity=20
- added joint rear_left_wheel_speed: type revolute, parent still_chassis_assm__list_nl250j021y5bmp_screwless, child wheel_assm__list_7stftxbui3bodm_screwless_3, origin xyz=-0.14849999999999990985 -1.249000902703301108e-16 -3.0531133177191804862e-16 rpy=3.1415926535897913396 6.1232339957475007072e-17 -1.5377205745436963724, axis 0 0 1, limit effort=1 velocity=20
- added joint rear_right_wheel_speed: type revolute, parent still_chassis_assm__list_nl250j021y5bmp_screwless, child wheel_assm__list_7stftxbui3bodm_screwless_4, origin xyz=-0.14849999999999960454 -1.1796119636642288242e-16 0.15600000000000030509 rpy=3.1415926535897913396 -5.6894649761932965311e-16 1.5377205745436963724, axis 0 0 1, limit effort=1 velocity=20
