Commit message: fix: repair mismatch between urdf joint names and fw published states

File: src/ballbot_description/urdf/ballbot.urdf (robot description, URDF)
Before this commit: robot ballbot_generated, 14 links, 13 joints
Joints:
- removed joint front_left_wheel_joint_speed
- removed joint front_right_wheel_joint_speed
- removed joint rear_left_wheel_joint_speed
- removed joint rear_right_wheel_joint_speed
- added joint front_left_wheel_joint: type continuous, parent still_chassis_assm, child wheel_assm, origin xyz=0.0680211 0.0783859 -0.0305 rpy=-1.5708 -1.4446e-29 9.71445e-17, axis 0 0 1, limit effort=10 velocity=10
- added joint front_right_wheel_joint: type continuous, parent still_chassis_assm, child wheel_assm_2, origin xyz=0.0680211 -0.0776141 -0.0305 rpy=-1.5708 -1.53772 -1.03884e-14, axis 0 0 1, limit effort=10 velocity=10
- added joint rear_left_wheel_joint: type continuous, parent still_chassis_assm, child wheel_assm_3, origin xyz=-0.0804789 0.0783859 -0.0305 rpy=-1.5708 1.5708 0, axis 0 0 1, limit effort=10 velocity=10
- added joint rear_right_wheel_joint: type continuous, parent still_chassis_assm, child wheel_assm_4, origin xyz=-0.0804789 -0.0776141 -0.0305 rpy=-1.5708 -1.53772 3.02617e-15, axis 0 0 1, limit effort=10 velocity=10
